File: mars-cm-carrier/mars-cm-carrier/mars-cm-carrier.kicad_pcb (KiCad board)
At the start: 2 copper layers, 170.2 x 170 mm, 77 parts, among them J2 USB3_A_Stacked, J7 Bus_M.2_Socket_M, J8 Bus_M.2_Socket_ECHANGEFOOTPRI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, J9 Bus_M.2_Socket_M, U1 Compute_Module_4_Connectors, U2 RT9742BNGJ5F, U3 ASM1184, U4 VL805, U5 W25Q32JVZP, Y1 25Mhz

Commit message: latest mars-cm-carrier ver
Parts:
- removed the J** at (132.1, 88.9)
- removed the REF** at (252.9, 175.0)
- removed the REF** at (129.2, 227.3)
- removed the REF** at (143.0, 227.3)
- removed the REF** at (159.8, 229.3)
- added J10: FRONT_PANEL_IO, Connector_PinSocket_2.54mm:PinSocket_2x05_P2.54mm_Vertical, B.Cu at (222.8, 225.1)
- added J11: USB2_FRONT_PANEL, Connector_PinSocket_2.54mm:PinSocket_2x05_P2.54mm_Vertical, F.Cu at (201.8, 227.9)
- added J12: Conn_02x10_Counter_Clockwise, Connector_PinSocket_2.54mm:PinSocket_2x10_P2.54mm_Vertical, F.Cu at (160.8, 225.7)
- added J13: 10018783-11200TLF, pciex16:10146070113Y0LF, F.Cu at (133.7, 123.1)
- moved C10 174.5 mm to (256.2, 198.4)
- moved C11 174.5 mm to (259.1, 182.7)
- moved C12 174.5 mm to (259.1, 184.6)
- moved C13 174.5 mm to (259.1, 186.6)
- moved C14 174.5 mm to (259.1, 188.6)
- moved C15 174.5 mm to (259.1, 190.6)
- moved C16 174.5 mm to (259.1, 192.5)
- moved C17 174.5 mm to (259.1, 194.5)
- moved C18 174.5 mm to (259.1, 196.5)
- moved C19 174.5 mm to (259.1, 198.4)
- moved C2 174.5 mm to (256.2, 182.7)
- moved C20 174.5 mm to (261.9, 182.7)
- moved C21 174.5 mm to (261.9, 184.6)
- moved C22 174.5 mm to (261.9, 186.6)
- moved C23 174.5 mm to (261.9, 188.6)
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Routing:
- net /PCIe_IN_TX_P: track 0.00 -> 0.81 mm
- net /PCIe_IN_TX_N: track 0.00 -> 0.78 mm
- added copper zone on B.Cu, net GND
- added copper zone on F.Cu, net GND
Other:
- copper layers 2 -> 6
