File: mars-cm-carrier/mars-cm-carrier/mars-cm-carrier.kicad_sch (KiCad schematic)
At the start: 73 parts, among them J1 HDMI_A, J2 USB3_A_Stacked, J3 USB_A_Stacked, J4 USB_C_Receptacle_USB2.0, J5 RJ45_LED, J6 Micro_SD_Card_Det2, J7 Bus_M.2_Socket_M, J8 Bus_M.2_Socket_ECHANGEFOOTPRI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, J9 Bus_M.2_Socket_M, U1 Compute_Module_4_Connectors, U2 RT9742BNGJ5F, U3 ASM1184, U4 VL805, U5 W25Q32JVZP, Y1 25Mhz

Commit message: latest mars-cm-carrier ver
Parts:
- added J10: FRONT_PANEL_IO, Connector_PinSocket_2.54mm:PinSocket_2x05_P2.54mm_Vertical, symbol Connector_Generic:Conn_02x05_Odd_Even
- added J11: USB2_FRONT_PANEL, Connector_PinSocket_2.54mm:PinSocket_2x05_P2.54mm_Vertical, symbol Connector_Generic:Conn_02x05_Odd_Even
- added J12: Conn_02x10_Counter_Clockwise, Connector_PinSocket_2.54mm:PinSocket_2x10_P2.54mm_Vertical, symbol Connector_Generic:Conn_02x10_Counter_Clockwise
- added J13: 10018783-11200TLF, CM4IO:PCIex1-36, symbol CM4IO:PCIe-x1
Connections:
- net +5V: now also J12.10 (Pin_10), J12.12 (Pin_12)
- net 5V: now also J10.9 (Pin_9), J11.1 (Pin_1), J11.2 (Pin_2)
- net GND: now also U1.107 (GND), U1.108 (GND), U1.113 (GND), U1.114 (GND), U1.119 (GND), U1.120 (GND), U1.125 (GND), U1.126 (GND), U1.131 (GND), U1.132 (GND), U1.137 (GND), U1.138 (GND), U1.144 (GND), U1.150 (GND), U1.155 (GND), U1.156 (GND), U1.161 (GND), U1.162 (GND), U1.167 (GND), U1.168 (GND), U1.173 (GND), U1.174 (GND), U1.179 (GND), U1.180 (GND), U1.185 (GND), U1.186 (GND), U1.191 (GND), U1.192 (GND), U1.197 (GND), U1.198 (GND), J11.7 (Pin_7), J11.8 (Pin_8), J12.15 (Pin_15), J12.18 (Pin_18), J12.4 (Pin_4), J12.7 (Pin_7), J13.A12 (GND), J13.A15 (GND), J13.A18 (GND), J13.A4 (GND), J13.B13 (GND), J13.B16 (GND), J13.B18 (GND), J13.B4 (GND), J13.B7 (GND)
- net PCIe_IN_RX_N: now also C29.2, U3.55 (TXN_IN)
- net PCIe_IN_RX_P: now also C28.2, U3.54 (TXP_IN)
- net USB2_D3+: now also J12.2 (Pin_2)
- net USB2_D3-: now also J12.3 (Pin_3)
- net USB2_D4+: now also J12.20 (Pin_20)
- net USB2_D4-: now also J12.19 (Pin_19)
- net USB3_RX3+: now also J12.8 (Pin_8)
- net USB3_RX3-: now also J12.9 (Pin_9)
- net USB3_RX4+: now also J12.14 (Pin_14)
- net USB3_RX4-: now also J12.13 (Pin_13)
- net USB3_TX3+: now also J12.5 (Pin_5)
- net USB3_TX4+: now also J12.17 (Pin_17)
- net USB3_TX4-: now also J12.16 (Pin_16)
- net USB_TX3-: now also J12.6 (Pin_6)
- new net +12v: J13.A2 (+12V), J13.A3 (+12V), J13.B1 (+12v), J13.B2 (+12v), J13.B3 (+12v)
- new net +3.3v: J13.A10 (+3.3V), J13.A5 (TCK), J13.A6 (TDI), J13.A8 (TMS), J13.A9 (+3.3V), J13.B10 (+3.3vAUX), J13.B8 (+3.3v), J13.B9 (nTRST)
- new net FPUSB_D+: J11.5 (Pin_5), J11.6 (Pin_6)
- new net FPUSB_D-: J11.3 (Pin_3), J11.4 (Pin_4)
- new net FP_USB_ID: J12.1 (Pin_1)
- new net HDLED+: J10.1 (Pin_1)
- new net HDLED-: J10.3 (Pin_3)
- new net NC: J11.10 (Pin_10)
- new net PCIeSOM_CLK_N: J13.A14 (REFCLK-)
- new net PCIeSOM_CLK_P: J13.A13 (REFCLK+)
- new net PCIeSOM_CLK_nREQ: J13.B12 (nCLKREQ)
- new net PCIeSOM_RX_N: J13.A16 (PERP0)
- new net PCIeSOM_RX_P: J13.A17 (PERN0)
- new net PCIeSOM_TX_N: J13.B14 (PETP0)
- new net PCIeSOM_TX_P: J13.B15 (PETN0)
- new net PCIeSOM_nRST: J13.A11 (nPERST)
- new net PLED+: J10.2 (Pin_2)
- new net PLED-: J10.4 (Pin_4)
- new net PWR+: J10.6 (Pin_6)
- new net PWR-: J10.8 (Pin_8)
- new net RST+: J10.5 (Pin_5)
- new net RST-: J10.7 (Pin_7)
- no-connect marks 4 -> 10
Other:
- moved on the sheet: R2, R3, R5, R7
