File: peltier-controller/peltier-controller/peltier-controller.kicad_sch (KiCad schematic)
At the start: 18 parts, among them J1 Peltier_Terminal, J2 Conn_01x03_Pin, J3 PWR_IN_15V, K1 SANYOU_SRD_Form_C, Q1 MJE3055, U1 ATtiny84A-SS, U2 AMS1117-3.3

Commit message: updated peltier
Parts:
- D1: footprint Diode_THT:D_DO-27_P15.24mm_Horizontal -> Diode_SMD:D_MELF
Changed lines of the file:
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@@
 			)
 		)
-		(property "Footprint" "Diode_THT:D_DO-27_P15.24mm_Horizontal"
+		(property "Footprint" "Diode_SMD:D_MELF"
 			(at 57.15 35.56 0)
 			(effects
