File: ccd-chromebook/ccd-chromebook/ccd-chromebook.kicad_sch (KiCad schematic)
At the start: 7 parts, among them J2 USB-C_2, P1 USB-C

Commit message: add updated files
Parts:
- added R1, R2: 68r, Resistor_SMD:R_0402_1005Metric, symbol Device:R
Connections:
- net DBG_N: now also R1.1; no longer J2.A7 (D-), J2.B7 (D-)
- net DBG_P: now also R2.1; no longer J2.A6 (D+), J2.B6 (D+)
- new net: J2.A7 (D-), J2.B7 (D-), R1.2
- new net: J2.A6 (D+), J2.B6 (D+), R2.2
