File: cm4-printing-deck/cm4-printing-deck/cm4-printing-deck.kicad_sch (KiCad schematic)
At the start: 200 parts, among them J1 Micro_SD_Card, J10 KB_USB, J2 USB_C_Receptacle_USB2.0_14P, J3 Reset, J4 debug, J5 Boot pins, J6 HDMI_A, J7 USB3_A, J8 USB3_A, J9 KB_USB, K1 KEYSW, K10 KEYSW, K11 KEYSW, K12 KEYSW, K13 KEYSW, K14 KEYSW, K15 KEYSW, K16 KEYSW, K17 KEYSW, K18 KEYSW, K19 KEYSW, K2 KEYSW, K20 KEYSW, K21 KEYSW, K22 KEYSW, K23 KEYSW, K24 KEYSW, K25 KEYSW, K26 KEYSW, K27 KEYSW, K28 KEYSW, K29 KEYSW, K3 KEYSW, K30 KEYSW, K31 KEYSW, K32 KEYSW, K33 KEYSW, K34 KEYSW, K35 KEYSW, K36 KEYSW, K37 KEYSW, K38 KEYSW, K39 KEYSW, K4 KEYSW, K40 KEYSW, K41 KEYSW, K42 KEYSW, K43 KEYSW, K44 KEYSW, K45 KEYSW, K46 KEYSW, K47 KEYSW, K48 KEYSW, K49 KEYSW, K5 KEYSW, K50 KEYSW, K51 KEYSW, K52 KEYSW, K53 KEYSW, K54 KEYSW, K55 KEYSW, K56 KEYSW, K57 KEYSW, K6 KEYSW, K60 KEYSW, K61 KEYSW, K7 KEYSW, K8 KEYSW, K9 KEYSW, SW20 Power, SW62 WIFIBT_DISABLE, U1 Compute_Module_4_Connectors, U10 AP2112K-3.3, U11 W25Q128JVS, U2 RP2040, U3 RT9742GGJ5, U5 PCF85063ATL, U6 74LVC1G07, U7 74LVC1G07, U8 74LVC1G07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

Commit message: minor routing and placement changes
Connections:
- net PCIe_RX_N is gone; now on net PE_RX_N: C17.1, U1.124 (PCIe_TX_N)
- net PCIe_RX_P is gone; now on net PE_RX_P: C18.1, U1.122 (PCIe_TX_P)
- net PCIe_CLK_N: no longer U1.112 (PCIe_CLK_N)
- net PCIe_CLK_P: no longer U1.110 (PCIe_CLK_P)
- net PCIe_CLK_nREQ: no longer U1.102 (~{PCIe_CLK_nREQ})
- net PCIe_TX_N: no longer U1.118 (PCIe_RX_N)
- net PCIe_TX_P: no longer U1.116 (PCIe_RX_P)
- net PCIe_nRST: no longer U1.109 (~{PCIe_nRST})
- net PE_RX_P: now reaches C18.2, U9.24 (PE_TXP)
- net PE_RX_N: now reaches C17.2, U9.25 (PE_TXN)
- new net PE_CLK_N: U1.112 (PCIe_CLK_N)
- new net PE_CLK_P: U1.110 (PCIe_CLK_P)
- new net PE_CLK_nREQ: U1.102 (~{PCIe_CLK_nREQ})
- new net PE_TX_N: U1.118 (PCIe_RX_N)
- new net PE_TX_P: U1.116 (PCIe_RX_P)
- new net PE_nRST: U1.109 (~{PCIe_nRST})
Other:
- moved on the sheet: C17, C18

Commit message: cm4-printing-deck: added fpc connectors for dsi panel
Parts:
- added C19, C20, C21: 0.1uF 10V, Capacitor_SMD:C_0402_1005Metric, symbol Device:C
- added C22: 22uF 6.3V, Capacitor_SMD:C_0402_1005Metric, symbol Device:C
- added C23, C24, C25, C27: 0.1uF 6.3V, Capacitor_SMD:C_0402_1005Metric, symbol Device:C
- added C26: 0.1uF 6V3, Capacitor_SMD:C_0603_1608Metric, symbol Device:C
- added C4: 22uF 10V, Capacitor_SMD:C_0402_1005Metric, symbol Device:C
- added J11: 3-2328724-1, moth:3-2328724-1, symbol cm4-panel-jdi-lt070me05000-rescue:3-2328724-1-Connector
- added J12: MOLEX_503480-0600, moth:screen_conn_2_nexus, symbol cm4-panel-jdi-lt070me05000-rescue:503480-0600-503480-0600
- added L1: BLM18TG121TN1D, Inductor_SMD:L_0603_1608Metric, symbol Device:L
- added R10, R19, R20, R21, R9: 10k 5%, Resistor_SMD:R_0402_1005Metric, symbol Device:R
- added U12: SN74LVC1G34DBVRG4, Package_TO_SOT_SMD:SOT-23-5, symbol cm4-panel-jdi-lt070me05000-rescue:SN74LVC1G34DBVRG4-Logic_LevelTranslator
- added U13: MCP23008T-E_SS, Package_SO:SSOP-20_5.3x7.2mm_P0.65mm, symbol cm4-panel-jdi-lt070me05000-rescue:MCP23008T-E_SS-MCP23008T-E_SS
Connections:
- net +3V3: now also C22.2, C23.2, C26.2, J11.26 (VDDp), J11.27 (VDDp), L1.2, R20.1, R21.1, U13.20 (VDD)
- net +5V: now also C19.2, C20.2, C21.2, C4.2, J11.1 (VDD), J11.2 (VDD), J11.3 (VDD), J11.4 (VDD)
- net GND: now also C19.1, C20.1, C21.1, C22.1, C23.1, C24.1, C25.1, C26.1, C27.1, C4.1, J11.11 (GND), J11.14 (GND), J11.17 (GND), J11.20 (GND), J11.23 (GND), J11.28 (GND), J11.29 (GND), J11.5 (GND), J11.8 (GND), J11.SH, J12.4, J12.S1 (SHIELD), J12.S2 (SHIELD), R10.2, R19.2, R9.1, U12.1 (NC), U12.3 (GND), U13.3 (A2), U13.4 (A1), U13.5 (A0), U13.9 (VSS)
- net SCL0: no longer U1.80 (I2C_SCL0)
- net SDA0: no longer U1.82 (I2C_SDA0)
- net MIPI_0_N: now reaches U1.175 (DSI1_D0_N)
- net MIPI_0_N: now also J11.12 (MIPI_0N)
- net MIPI_0_P: now reaches U1.177 (DSI1_D0_P)
- net MIPI_0_P: now also J11.13 (MIPI_0P)
- net MIPI_1_N: now reaches U1.181 (DSI1_D1_N)
- net MIPI_1_N: now also J11.18 (MIPI_1N)
- net MIPI_1_P: now reaches U1.183 (DSI1_D1_P)
- net MIPI_1_P: now also J11.19 (MIPI_1P)
- net MIPI_CLK_N: now reaches U1.187 (DSI1_C_N)
- net MIPI_CLK_N: now also J11.15 (MIPI_CLKN)
- net MIPI_CLK_P: now reaches U1.189 (DSI1_C_P)
- net MIPI_CLK_P: now also J11.16 (MIPI_CLKP)
- net MIPI_2_N: now reaches U1.193 (DSI1_D2_N)
- net MIPI_2_N: now also J11.21 (MIPI_2N)
- net MIPI_3_N: now reaches U1.194 (DSI1_D3_N)
- net MIPI_3_N: now also J11.9 (MIPI_3N)
- net MIPI_2_P: now reaches U1.195 (DSI1_D2_P)
- net MIPI_2_P: now also J11.22 (MIPI_2P)
- net MIPI_3_P: now reaches U1.196 (DSI1_D3_P)
- net MIPI_3_P: now also J11.10 (MIPI_3P)
- new net: R20.2, U13.6 (*RESET)
- new net: C27.2, J12.1, L1.1
- new net: J11.24 (XRES), U12.4 (Y)
- new net +1V8: C24.2, C25.2, J11.31 (IOVCC), U12.5 (VCC)
- new net BL_CNTRL: J11.6 (LED_EN), R10.1, U13.16 (GP4)
- new net EXP_INT: R21.2, U13.8 (INT)
- new net EXP_P2: U13.14 (GP2)
- new net LCD_PWR_EN: J11.30 (DCDC_EN), R9.2, U13.17 (GP5)
- new net LCD_RESET: R19.1, U12.2 (A), U13.15 (GP3)
- new net SCL: J12.6, U1.80 (I2C_SCL0), U13.1 (SCL)
- new net SDA: J12.5, U1.82 (I2C_SDA0), U13.2 (SDA)
- new net TOUCH_INT: J12.2, U13.13 (GP1)
- new net TOUCH_RST: J12.3, U13.12 (GP0)
- no-connect marks 138 -> 136

Commit message: cm4-printing-deck: layout changes, LCD connector + associated added, slight routing changes. moved keyboard to separate project
Parts:
- removed C10, C11, C12, C13, C14, C7, C8, C9: 1uF, Capacitor_SMD:C_0603_1608Metric, symbol Device:C
- removed C3: 0.1uF, Capacitor_SMD:C_0603_1608Metric, symbol Device:C
- removed C5, C6: 27pF, Capacitor_SMD:C_0603_1608Metric, symbol Device:C
- removed D10, D11, D12, D13, D14, D15, D16, D17, D18, D19, D20, D21, D22, D23, D25, D26, D29, D3, D30, D31, D32, D33, D34, D35, D36, D37, D38, D39, D4, D40, D41, D42, D43, D44, D45, D46, D47, D48, D49, D5, D50, D51, D52, D53, D54, D55, D56, D57, D58, D59, D6, D60, D61, D62, D65, D66, D7, D8, D9: D, Diode_SMD:D_SOD-123, symbol Device:D
- removed J3: Reset, Connector_PinHeader_2.54mm:PinHeader_1x02_P2.54mm_Vertical, symbol Connector:Conn_01x02_Pin
- removed J4: debug, Connector_PinHeader_1.27mm:PinHeader_1x03_P1.27mm_Vertical, symbol Connector:Conn_01x03_Pin
- removed J5: Boot pins, Connector_PinHeader_2.54mm:PinHeader_1x02_P2.54mm_Vertical, symbol Connector:Conn_01x02_Pin
- removed J9: KB_USB, Connector_PinHeader_2.54mm:PinHeader_1x04_P2.54mm_Vertical, symbol Connector_Generic:Conn_01x04
- removed K1, K10, K11, K12, K13, K14, K15, K16, K17, K18, K19, K2, K20, K21, K22, K23, K24, K25, K26, K27, K28, K29, K3, K30, K31, K32, K33, K34, K35, K36, K37, K38, K39, K4, K40, K41, K42, K43, K44, K45, K46, K47, K48, K49, K5, K50, K51, K52, K53, K54, K55, K56, K57, K6, K60, K61, K7, K8, K9: KEYSW, Button_Switch_SMD:SW_SPST_PTS645, symbol keyboard_parts:KEYSW
- removed R11: DNP, Resistor_SMD:R_0603_1608Metric, symbol Device:R
- removed R12, R7: 1k, Resistor_SMD:R_0603_1608Metric, symbol Device:R
- removed R13, R14: 27r, Resistor_SMD:R_0603_1608Metric, symbol Device:R
- removed R15, R8: 10k, Resistor_SMD:R_0603_1608Metric, symbol Device:R
- removed U10: AP2112K-3.3, Package_TO_SOT_SMD:SOT-23-5, symbol Regulator_Linear:AP2112K-3.3
- removed U11: W25Q128JVS, Package_SO:SOIC-8_5.23x5.23mm_P1.27mm, symbol Memory_Flash:W25Q128JVS
- removed U2: RP2040, Package_DFN_QFN:QFN-56-1EP_7x7mm_P0.4mm_EP3.2x3.2mm, symbol MCU_RaspberryPi:RP2040
- removed Y1: 12MHz, Crystal:Crystal_SMD_3215-2Pin_3.2x1.5mm, symbol Device:Crystal
- added U14: AP1117-18, Package_TO_SOT_SMD:SOT-223-3_TabPin2, symbol Regulator_Linear:AP1117-18
- C19, C20, C21: value 0.1uF 10V -> 0.1uF
- C22: value 22uF 6.3V -> 22uF
- C23, C24, C25, C27: value 0.1uF 6.3V -> 0.1uF
- C26: value 0.1uF 6V3 -> 0.1uF
- C4: value 22uF 10V -> 22uF
- R10, R19, R20, R21, R9: value 10k 5% -> 10k
Connections:
- net +1V8: now also U14.2 (VO)
- net +5V: now also U14.3 (VI)
- net GND: now also U14.1 (GND)
- no-connect marks 136 -> 132

Commit message: cm4-printing-deck: updated silkscreen
Parts:
- removed BT1: BAT1, Connector_PinSocket_2.54mm:PinSocket_1x02_P2.54mm_Horizontal, symbol Device:Battery_Cell
- removed C1, C2: 10uf, Capacitor_SMD:C_0603_1608Metric, symbol Device:C
- removed D1: GREEN_CHRG, LED_SMD:LED_0805_2012Metric, symbol Device:LED
- removed D2: RED_CHRG, LED_SMD:LED_0805_2012Metric, symbol Device:LED
- removed R3: R, Resistor_SMD:R_0603_1608Metric, symbol Device:R
- removed R4, R5: 1k, Resistor_SMD:R_0603_1608Metric, symbol Device:R
- removed R6: 1.2k, Resistor_SMD:R_0603_1608Metric, symbol Device:R
- removed TP1: TP4056, Package_SO:SOP-8_6.605x9.655mm_P2.54mm, symbol moth_library:TP4056
- removed U4: ~, Package_TO_SOT_SMD:SOT-223, symbol RT9742GGJ5:RT9742SNGV
- added C10, C11, C12, C13, C3, C5, C6, C7, C8, C9: 10u, Capacitor_SMD:C_0603_1608Metric, symbol Device:C
- added C14, C30: 100n, Capacitor_SMD:C_0603_1608Metric, symbol Device:C
- added C28: 10n, Capacitor_SMD:C_0603_1608Metric, symbol Device:C
- added C29: 1.2n, Capacitor_SMD:C_0603_1608Metric, symbol Device:C
- added C31: 100uF, Capacitor_SMD:CP_Elec_4x4.5, symbol Device:C_Polarized
- added C32, C33: 10uF, Capacitor_SMD:C_0402_1005Metric, symbol Device:C
- added C34, C39: 1uF, Capacitor_SMD:C_0402_1005Metric, symbol Device:C
- added J3: PWR_BAT, Connector_PinHeader_2.54mm:PinHeader_1x04_P2.54mm_Vertical, symbol Connector:Conn_01x04_Pin
- added L2: SRN6045TA-3R3Y, SRN6045TA_3R3Y:IND_SRN6045TA-3R3Y, symbol SRN6045TA-3R3Y:SRN6045TA-3R3Y
- added R7: 20k, Resistor_SMD:R_0603_1608Metric, symbol Device:R
- added U10: CH32X05, Package_SO:TSSOP-20_4.4x6.5mm_P0.65mm, symbol CH32X035F7P6:CH32X035F7P6_me
- added U11: AP2112K-3.3, Package_TO_SOT_SMD:SOT-23-5, symbol Regulator_Linear:AP2112K-3.3
- added U2: AP64501SP-13, Package_SO:Diodes_SO-8EP, symbol AP64501SP:AP64501SP-13
- added U4: TPS784105QWDRBRQ1, Package_SON:SON-8-1EP_3x2mm_P0.5mm_EP1.4x1.6mm, symbol TPS784105QWDRBRQ1:TPS784105QWDRBRQ1
- C17, C18: footprint Capacitor_SMD:C_0603_1608Metric -> Capacitor_SMD:C_0402_1005Metric
- C19, C21, C24: value 0.1uF -> 0.1uF
- J7: footprint Connector_USB:USB3_A_Receptacle_Wuerth_692122030100 -> Connector_USB:USB_C_Receptacle_CNCTech_C-ARA1-AK51X; symbol Connector:USB3_A -> Connector:USB_C_Receptacle
- R1: value 5.6k -> 10r
- R2: value 5.6k -> 20k
Connections:
- net HDMI_5V is gone; now on net +5V: J6.18 (+5V)
- net PCIe_CLK_N is gone; now on net PE_CLK_N: U9.22 (PE_CLKN)
- net PCIe_CLK_P is gone; now on net PE_CLK_P: U9.21 (PE_CLKP)
- net PCIe_CLK_nREQ is gone; now on net PE_CLK_nREQ: U9.30 (~{PE_CLKREQ})
- net PCIe_TX_N is gone; now on net PE_TX_N: U9.28 (PE_RXN)
- net PCIe_TX_P is gone; now on net PE_TX_P: U9.27 (PE_RXP)
- net PCIe_nRST is gone; now on net PE_nRST: U9.19 (~{PE_RST})
- net SCL0 is gone; now on net SCL: U5.7 (SCL)
- net SDA0 is gone; now on net SDA: U5.6 (SDA)
- net +3V3: now also U14.3 (VI), C39.1, U11.5 (VOUT); no longer U1.84 (CM4_3.3V_Out), U1.86 (CM4_3.3V_Out)
- net +5V: now also J7.A4 (VBUS), J7.A9 (VBUS), J7.B4 (VBUS), J7.B9 (VBUS), J8.1 (VBUS), R2.2, C10.1, C11.1, C12.1, C13.1, C31.1, C32.2, C34.1, J3.3 (Pin_3), J3.4 (Pin_4), L2.2, U10.15 (VDD), U11.1 (VIN), U11.3 (EN), U2.5 (FB), U4.6 (EN), U4.8 (IN); no longer J2.A4 (VBUS), J2.A9 (VBUS), J2.B4 (VBUS), J2.B9 (VBUS), U14.3 (VI)
- net 1.05v: now also C33.2, U4.1 (OUT)
- net BL_CNTRL: now also U13.17 (GP5); no longer U13.16 (GP4)
- net GND: now also J7.A1 (GND), J7.A12 (GND), J7.B1 (GND), J7.B12 (GND), J7.S1 (SHIELD), R2.1, C10.2, C11.2, C12.2, C13.2, C28.2, C29.2, C3.2, C30.2, C31.2, C32.1, C33.1, C34.2, C39.2, C5.2, C6.2, C7.2, C8.2, C9.2, J3.1 (Pin_1), J3.2 (Pin_2), L2.1, U10.16 (GND), U11.2 (GND), U2.7 (GND), U2.8 (SW), U2.EPAD (GND), U4.5 (GND), U4.9 (PAD); no longer J7.10 (SHIELD), J7.4 (GND), J7.7 (DRAIN), R2.2
- net LCD_PWR_EN: now also U13.15 (GP3); no longer U13.17 (GP5)
- net LCD_RESET: now also U13.16 (GP4); no longer U13.15 (GP3)
- net PE_RX_N: no longer C17.2, U9.25 (PE_TXN)
- net PE_RX_P: no longer C18.2, U9.24 (PE_TXP)
- net SCL: now also U10.20 (SCK/PA5)
- net SDA: now also U10.19 (MISO/PA6)
- net SSRX1+: now also J7.B11 (RX1+); no longer J7.6 (SSRX+)
- net SSRX1-: now also J7.B10 (RX1-); no longer J7.5 (SSRX-)
- net SSRX2+: now also J7.A11 (RX2+); no longer J8.6 (SSRX+)
- net SSRX2-: now also J7.A10 (RX2-); no longer J8.5 (SSRX-)
- net SSTX1+: now also J7.A2 (TX1+); no longer J7.9 (SSTX+)
- net SSTX1-: now also J7.A3 (TX1-); no longer J7.8 (SSTX-)
- net SSTX2+: now also J7.B2 (TX2+); no longer J8.9 (SSTX+)
- net SSTX2-: now also J7.B3 (TX2-); no longer J8.8 (SSTX-)
- net USB2D1+: now also J7.A6 (D+), J7.B6 (D+); no longer J7.3 (D+)
- net USB2D1-: now also J7.A7 (D-), J7.B7 (D-); no longer J7.2 (D-)
- net SSTX3+: now reaches U9.1 (SSTX3+)
- net SSTX3+: now also J8.9 (SSTX+)
- net SSTX3-: now reaches U9.2 (SSTX3-)
- net SSTX3-: now also J8.8 (SSTX-)
- net SSRX3+: now reaches U9.4 (SSRX3+)
- net SSRX3+: now also J8.6 (SSRX+)
- net SSRX3-: now reaches U9.5 (SSRX3-)
- net SSRX3-: now also J8.5 (SSRX-)
- net USB2D3+: now reaches U9.7 (USB2D3+)
- net USB2D3-: now reaches U9.8 (USB2D3-)
- net at R1.1: now also C14.1; no longer J2.A5 (CC1)
- net CH32_USB_P: now reaches J2.A6 (D+)
- net CH32_USB_P: now also J2.B6 (D+), U10.13 (UPD/PC17)
- net CH32_USB_N: now reaches J2.A7 (D-)
- net CH32_USB_N: now also J2.B7 (D-), U10.14 (UDM/PC16)
- net CC2: now reaches J2.B5 (CC2)
- net CC2: now also U10.3 (PC15/CC2); no longer R2.1
- new net: C29.1, R7.1
- new net: C28.1, R7.2, U2.6 (COMP)
- new net: C14.2, U2.1 (BST)
- new net: C30.1, U2.4 (SS)
- new net CC1: J2.A5 (CC1), U10.2 (PC14/CC1)
- new net PE_RX_C_N: C17.2, U9.25 (PE_TXN)
- new net PE_RX_C_P: C18.2, U9.24 (PE_TXP)
- new net VBUS: C3.1, C5.1, C6.1, C7.1, C8.1, C9.1, J2.A4 (VBUS), J2.A9 (VBUS), J2.B4 (VBUS), J2.B9 (VBUS), U2.2 (VIN), U2.3 (EN)
- no-connect marks 132 -> 142
Other:
- moved on the sheet: C25, C27, J8, L1, R19

Commit message: add updated files
Connections:
- net +5V: now also U10.1 (VDD); no longer U10.15 (VDD)
- net CC1: now also U10.19 (PC14/CC2); no longer U10.2 (PC14/CC1)
- net CC2: now also U10.20 (PC15/CC2); no longer U10.3 (PC15/CC2)
- net CH32_USB_N: now also U10.17 (PC16); no longer U10.14 (UDM/PC16)
- net CH32_USB_P: now also U10.18 (PC17); no longer U10.13 (UPD/PC17)
- net GND: no longer U10.16 (GND)
- net SCL: no longer U10.20 (SCK/PA5)
- net SDA: no longer U10.19 (MISO/PA6)
- no-connect marks 142 -> 139
