File: simple-rp235x/simple-rp235x/simple-rp235x.kicad_pcb (KiCad board)
At the start: 2 copper layers, 59 x 21.5 mm, 46 parts, among them J1 USB_C_Receptacle, J2 GPIO_1, J3 GPIO_2, J4 Conn_01x02_Pin, SW1 RUN, SW2 USB_BOOT, U2 FUSB302B01MPX, U3 AP2112K-3.3, U4 W25Q32JVSS, Y1 12MHz

Commit message: add updated files
Parts:
- moved C12 0.68 mm to (102.7, 64.3), turned to -45 degrees
- moved C10 0.07 mm to (113.0, 71.3)
Routing:
- net 1V1_C: track 34.8 -> 36.5 mm
- net GPIO47_VBUS_ADC: track 39.0 -> 38.5 mm
