File: tiny-ccd/tiny-ccd/tiny-ccd.kicad_pcb (KiCad board)
At the start: 2 copper layers, 21.1 x 15.2 mm, 10 parts, among them J1 USB-C_PLUG, J2 USB-C_DEBUG, J3 USB-C_DATA

Commit message: add updated files
Parts:
- added R2: 68r, Resistor_SMD:R_0402_1005Metric, F.Cu at (149.4, 105.0)
- added R5: 68r, Resistor_SMD:R_0402_1005Metric, F.Cu at (150.5, 105.0)
- J2: value USB-C_DEBUG -> USB-C_DATA
- J3: value USB-C_DATA -> USB-C_DEBUG; moved to B.Cu
- moved R4 3.11 mm to (160.6, 101.6)
- moved D2 0.58 mm to (147.4, 102.7)
- moved R1 0.55 mm to (148.4, 103.5)
- moved J2 0.14 mm to (149.8, 111.4)
- turned J3 to 180 degrees
Connections:
- J2 pad A6: USB_P -> Net-(J2-D+-PadA6)
- J2 pad A7: USB_N -> Net-(J2-D--PadA7)
- J2 pad B6: USB_P -> Net-(J2-D+-PadA6)
- J2 pad B7: USB_N -> Net-(J2-D--PadA7)
Routing:
- net Net-(J2-D--PadA7): track 0.00 -> 4.94 mm
- net Net-(J2-D+-PadA6): track 0.00 -> 4.82 mm
- net USB_N: track 17.3 -> 13.2 mm
- net USB_P: track 15.7 -> 11.9 mm
- net CC2: track 3.54 -> 6.67 mm
- net DBG_P: track 14.5 -> 11.6 mm, vias 1 -> 0
- net VBUS: track 47.8 -> 49.7 mm
- net DBG_N: track 14.0 -> 13.1 mm, vias 2 -> 1
- net GND: vias 10 -> 14
