File: tiny-ccd/tiny-ccd/tiny-ccd.kicad_sch (KiCad schematic)
At the start: 10 parts, among them J2 USB-C_DEBUG, J3 USB-C_DATA, P1 USB-C_PLUG

Commit message: add updated files
Parts:
- added R2, R5: 68r, Resistor_SMD:R_0402_1005Metric, symbol Device:R
- J2: value USB-C_DEBUG -> USB-C_DATA
- J3: value USB-C_DATA -> USB-C_DEBUG
Connections:
- net USB_N: now also R2.2; no longer J2.A7 (D-), J2.B7 (D-)
- net USB_P: now also R5.1; no longer J2.A6 (D+), J2.B6 (D+)
- new net: J2.A6 (D+), J2.B6 (D+), R5.2
- new net: J2.A7 (D-), J2.B7 (D-), R2.1
Other:
- moved on the sheet: C1, C2
