File: usb-uart-eqmod/usb-uart-eqmod/usb-uart-eqmod.kicad_pcb (KiCad board)
At the start: 2 copper layers, 48.9 x 21.5 mm, 25 parts, among them J1 USB_C_Receptacle_USB2.0_14P, J2 RJ45, U1 FT232RL, U2 ADuM1200AR, U3 L78L05_SOT89

Commit message: minor routing and placement changes
Parts:
- moved D1 2.29 mm to (123.3, 86.8), turned to 90 degrees
- moved R1 0.88 mm to (121.5, 86.7), turned to 90 degrees
- moved R3 0.77 mm to (146.9, 77.5)
- moved R2 0.72 mm to (145.5, 77.5)
- moved R7 0.16 mm to (120.0, 86.7)
Routing:
- net Net-(U1-VCC): track 34.8 -> 33.3 mm
- net Net-(U3-IN): track 24.4 -> 23.1 mm
- net Net-(D1-A): track 1.51 -> 2.43 mm
- net Net-(D3-A): track 11.8 -> 11.0 mm
- net Net-(J2-Pad5): track 20.0 -> 19.3 mm
Other:
- board text added: "moth :)"
- board text removed: "designed by moth"
