File: d2000-mitx/d2000-mitx/01_block.kicad_sch (KiCad schematic)
At the start: 0 parts

Commit message: update schem + pcb layout
Parts:
- added H1, H2, H3, H4, H5, H6: MountingHole, MountingHole:MountingHole_3.2mm_M3_Pad, symbol Mechanical:MountingHole
Other:
- note added: "PCIe to USB VL805 (Rear)"
- note added: "RP2040 (EC duties)"
- note removed: "CPLD"
- note removed: "M.2 PCIe 3.0 4x"
- note removed: "PCIe Gen3 X2"
