File: d2000-mitx/d2000-mitx/03_D2000.kicad_sch (KiCad schematic)
At the start: 5 parts

Commit message: update schem + pcb layout
Parts:
- removed U3: ~, D2000:D2000_DDR4_BGA1144P100_3500X350, symbol D2000-FT20004:D2000-E8
- added U5: ~, D2000:D2000_DDR4_BGA1144P100_3500X350, symbol D2000-FT20004:D2000-E8
Connections:
- net FT_MEM0_A0: now also U5.B28 (LMU0_A0)
- net FT_MEM0_A1: now also U5.F25 (LMU0_A1)
- net FT_MEM0_A10: now also U5.D28 (LMU0_A10)
- net FT_MEM0_A11: now also U5.E24 (LMU0_A11)
- net FT_MEM0_A12: now also U5.B23 (LMU0_A12)
- net FT_MEM0_A13: now also U5.B29 (LMU0_A13)
- net FT_MEM0_A14: now also U5.G27 (LMU0_A14/WE_N)
- net FT_MEM0_A15: now also U5.H27 (LMU0_A15/CAS_N)
- net FT_MEM0_A16: now also U5.H26 (LMU0_A16/RAS_N)
- net FT_MEM0_A17: now also U5.A31 (LMU0_A17)
- net FT_MEM0_A2: now also U5.G25 (LMU0_A2)
- net FT_MEM0_A3: now also U5.A25 (LMU0_A3)
- net FT_MEM0_A4: now also U5.B25 (LMU0_A4)
- net FT_MEM0_A5: now also U5.C25 (LMU0_A5)
- net FT_MEM0_A6: now also U5.F23 (LMU0_A6)
- net FT_MEM0_A7: now also U5.D24 (LMU0_A7)
- net FT_MEM0_A8: now also U5.C24 (LMU0_A8)
- net FT_MEM0_A9: now also U5.A23 (LMU0_A9)
- net FT_MEM0_ACT_N: now also U5.F22 (LMU0_ACT_N)
- net FT_MEM0_ALERT_N: now also U5.G22 (LMU0_BP_ALERT_N)
- net FT_MEM0_BA0: now also U5.G26 (LMU0_BA0)
- net FT_MEM0_BA1: now also U5.C28 (LMU0_BA1)
- net FT_MEM0_BG0: now also U5.E23 (LMU0_BG0)
- net FT_MEM0_BG1: now also U5.E22 (LMU0_BG1)
- net FT_MEM0_C0: now also U5.D30 (LMU0_C0)
- net FT_MEM0_C1: now also U5.C31 (VSS)
- net FT_MEM0_C2: now also U5.B32 (VSS)
- net FT_MEM0_CKE0: now also U5.B22 (LMU0_CKE0)
- net FT_MEM0_CKE1: now also U5.D22 (LMU0_CKE1)
- net FT_MEM0_CLK0_C: now also U5.E25 (LMU0_CLK_C0)
- net FT_MEM0_CLK0_T: now also U5.D25 (LMU0_CLK_T0)
- net FT_MEM0_CLK1_C: now also U5.F26 (LMU0_CLK_C1)
- net FT_MEM0_CLK1_T: now also U5.E26 (LMU0_CLK_T1)
- net FT_MEM0_CS_N0: now also U5.E28 (LMU0_CS0)
- net FT_MEM0_CS_N1: now also U5.B31 (LMU0_CS1)
- net FT_MEM0_DQ0: now also U5.L32 (LMU0_DQ0)
- net FT_MEM0_DQ1: now also U5.L34 (LMU0_DQ1)
- net FT_MEM0_DQ10: now also U5.U32 (LMU0_DQ10)
- net FT_MEM0_DQ11: now also U5.U31 (LMU0_DQ11)
- net FT_MEM0_DQ12: now also U5.P34 (LMU0_DQ12)
- net FT_MEM0_DQ13: now also U5.T32 (LMU0_DQ13)
- net FT_MEM0_DQ14: now also U5.U34 (LMU0_DQ14)
- net FT_MEM0_DQ15: now also U5.P32 (LMU0_DQ15)
- net FT_MEM0_DQ16: now also U5.D33 (LMU0_DQ16)
- net FT_MEM0_DQ17: now also U5.G32 (LMU0_DQ17)
- net FT_MEM0_DQ18: now also U5.G33 (LMU0_DQ18)
- net FT_MEM0_DQ19: now also U5.D34 (LMU0_DQ19)
- net FT_MEM0_DQ2: now also U5.P31 (LMU0_DQ2)
- net FT_MEM0_DQ20: now also U5.D32 (LMU0_DQ20)
- net FT_MEM0_DQ21: now also U5.F31 (LMU0_DQ21)
- net FT_MEM0_DQ22: now also U5.F33 (LMU0_DQ22)
- net FT_MEM0_DQ23: now also U5.C33 (LMU0_DQ23)
- net FT_MEM0_DQ24: now also U5.G34 (LMU0_DQ24)
- net FT_MEM0_DQ25: now also U5.K31 (LMU0_DQ25)
- net FT_MEM0_DQ26: now also U5.K32 (LMU0_DQ26)
- net FT_MEM0_DQ27: now also U5.H30 (LMU0_DQ27)
- net FT_MEM0_DQ28: now also U5.H29 (LMU0_DQ28)
- net FT_MEM0_DQ29: now also U5.G30 (LMU0_DQ29)
- net FT_MEM0_DQ3: now also U5.N32 (LMU0_DQ3)
- net FT_MEM0_DQ30: now also U5.J33 (LMU0_DQ30)
- net FT_MEM0_DQ31: now also U5.J31 (LMU0_DQ31)
- net FT_MEM0_DQ32: now also U5.A14 (LMU0_DQ32)
- net FT_MEM0_DQ33: now also U5.B17 (LMU0_DQ33)
- net FT_MEM0_DQ34: now also U5.A17 (LMU0_DQ34)
- net FT_MEM0_DQ35: now also U5.B14 (LMU0_DQ35)
- net FT_MEM0_DQ36: now also U5.D14 (LMU0_DQ36)
- net FT_MEM0_DQ37: now also U5.C17 (LMU0_DQ37)
- net FT_MEM0_DQ38: now also U5.A16 (LMU0_DQ38)
- net FT_MEM0_DQ39: now also U5.C14 (LMU0_DQ39)
- net FT_MEM0_DQ4: now also U5.K34 (LMU0_DQ4)
- net FT_MEM0_DQ40: now also U5.G17 (LMU0_DQ40)
- net FT_MEM0_DQ41: now also U5.F20 (LMU0_DQ41)
- net FT_MEM0_DQ42: now also U5.E21 (LMU0_DQ42)
- net FT_MEM0_DQ43: now also U5.G16 (LMU0_DQ43)
- net FT_MEM0_DQ44: now also U5.F16 (LMU0_DQ44)
- net FT_MEM0_DQ45: now also U5.E16 (LMU0_DQ45)
- net FT_MEM0_DQ46: now also U5.G20 (LMU0_DQ46)
- net FT_MEM0_DQ47: now also U5.D19 (LMU0_DQ47)
- net FT_MEM0_DQ48: now also U5.A10 (LMU0_DQ48)
- net FT_MEM0_DQ49: now also U5.C11 (LMU0_DQ49)
- net FT_MEM0_DQ5: now also U5.L33 (LMU0_DQ5)
- net FT_MEM0_DQ50: now also U5.B13 (LMU0_DQ50)
- net FT_MEM0_DQ51: now also U5.A13 (LMU0_DQ51)
- net FT_MEM0_DQ52: now also U5.E10 (LMU0_DQ52)
- net FT_MEM0_DQ53: now also U5.D10 (LMU0_DQ53)
- net FT_MEM0_DQ54: now also U5.C13 (LMU0_DQ54)
- net FT_MEM0_DQ55: now also U5.A12 (LMU0_DQ55)
- net FT_MEM0_DQ56: now also U5.G12 (LMU0_DQ56)
- net FT_MEM0_DQ57: now also U5.F15 (LMU0_DQ57)
- net FT_MEM0_DQ58: now also U5.E15 (LMU0_DQ58)
- net FT_MEM0_DQ59: now also U5.G11 (LMU0_DQ59)
- net FT_MEM0_DQ6: now also U5.N33 (LMU0_DQ6)
- net FT_MEM0_DQ60: now also U5.G10 (LMU0_DQ60)
- net FT_MEM0_DQ61: now also U5.F10 (LMU0_DQ61)
- net FT_MEM0_DQ62: now also U5.G13 (LMU0_DQ62)
- net FT_MEM0_DQ63: now also U5.G14 (LMU0_DQ63)
- net FT_MEM0_DQ64: now also U5.A18 (LMU0_CB0)
- net FT_MEM0_DQ65: now also U5.A21 (LMU0_CB1)
- net FT_MEM0_DQ66: now also U5.D21 (LMU0_CB2)
- net FT_MEM0_DQ67: now also U5.B18 (LMU0_CB3)
- net FT_MEM0_DQ68: now also U5.D17 (LMU0_CB4)
- net FT_MEM0_DQ69: now also U5.B20 (LMU0_CB5)
- net FT_MEM0_DQ7: now also U5.N34 (LMU0_DQ7)
- net FT_MEM0_DQ70: now also U5.D18 (LMU0_CB6)
- net FT_MEM0_DQ71: now also U5.A20 (LMU0_CB7)
- net FT_MEM0_DQ8: now also U5.R34 (LMU0_DQ8)
- net FT_MEM0_DQ9: now also U5.R33 (LMU0_DQ9)
- net FT_MEM0_DQS_C_0: now also U5.M34 (LMU0_DQS_C0)
- net FT_MEM0_DQS_C_1: now also U5.T34 (LMU0_DQS_C1)
- net FT_MEM0_DQS_C_10: now also U5.T31 (LMU0_DQS_C10)
- net FT_MEM0_DQS_C_11: now also U5.E32 (LMU0_DQS_C11)
- net FT_MEM0_DQS_C_12: now also U5.H32 (LMU0_DQS_C12)
- net FT_MEM0_DQS_C_13: now also U5.A15 (LMU0_DQS_C13)
- net FT_MEM0_DQS_C_14: now also U5.E18 (LMU0_DQS_C14)
- net FT_MEM0_DQS_C_15: now also U5.A11 (LMU0_DQS_C15)
- net FT_MEM0_DQS_C_16: now also U5.E12 (LMU0_DQS_C16)
- net FT_MEM0_DQS_C_17: now also U5.A19 (LMU0_DQS_C17)
- net FT_MEM0_DQS_C_2: now also U5.E34 (LMU0_DQS_C2)
- net FT_MEM0_DQS_C_3: now also U5.H34 (LMU0_DQS_C3)
- net FT_MEM0_DQS_C_4: now also U5.D15 (LMU0_DQS_C4)
- net FT_MEM0_DQS_C_5: now also U5.F19 (LMU0_DQS_C5)
- net FT_MEM0_DQS_C_6: now also U5.D11 (LMU0_DQS_C6)
- net FT_MEM0_DQS_C_7: now also U5.E13 (LMU0_DQS_C7)
- net FT_MEM0_DQS_C_8: now also U5.C19 (LMU0_DQS_C8)
- net FT_MEM0_DQS_C_9: now also U5.M31 (LMU0_DQS_C9)
- net FT_MEM0_DQS_T_0: now also U5.M33 (LMU0_DQS_T0)
- net FT_MEM0_DQS_T_1: now also U5.T33 (LMU0_DQS_T1)
- net FT_MEM0_DQS_T_10: now also U5.R31 (LMU0_DQS_T10)
- net FT_MEM0_DQS_T_11: now also U5.E31 (LMU0_DQS_T11)
- net FT_MEM0_DQS_T_12: now also U5.H31 (LMU0_DQS_T12)
- net FT_MEM0_DQS_T_13: now also U5.B15 (LMU0_DQS_T13)
- net FT_MEM0_DQS_T_14: now also U5.F18 (LMU0_DQS_T14)
- net FT_MEM0_DQS_T_15: now also U5.B11 (LMU0_DQS_T15)
- net FT_MEM0_DQS_T_16: now also U5.F12 (LMU0_DQS_T16)
- net FT_MEM0_DQS_T_17: now also U5.B19 (LMU0_DQS_T17)
- net FT_MEM0_DQS_T_2: now also U5.F34 (LMU0_DQS_T2)
- net FT_MEM0_DQS_T_3: now also U5.J34 (LMU0_DQS_T3)
- net FT_MEM0_DQS_T_4: now also U5.D16 (LMU0_DQS_T4)
- net FT_MEM0_DQS_T_5: now also U5.E19 (LMU0_DQS_T5)
- net FT_MEM0_DQS_T_6: now also U5.D12 (LMU0_DQS_T6)
- net FT_MEM0_DQS_T_7: now also U5.D13 (LMU0_DQS_T7)
- net FT_MEM0_DQS_T_8: now also U5.C20 (LMU0_DQS_T8)
- net FT_MEM0_DQS_T_9: now also U5.L31 (LMU0_DQS_T9)
- net FT_MEM0_ODT0: now also U5.G28 (LMU0_ODT0)
- net FT_MEM0_ODT1: now also U5.F29 (LMU0_ODT1)
- net FT_MEM0_PAR: now also U5.A28 (LMU0_PAR)
- net FT_MEM0_RST_N: now also U5.H22 (LMU0_BP_MEMRESET_L)
- net FT_MEM1_A0: now also U5.AN28 (LMU1_A0)
- net FT_MEM1_A1: now also U5.AJ25 (LMU1_A1)
- net FT_MEM1_A10: now also U5.AL28 (LMU1_A10)
- net FT_MEM1_A11: now also U5.AK24 (LMU1_A11)
- net FT_MEM1_A12: now also U5.AN23 (LMU1_A12)
- net FT_MEM1_A13: now also U5.AN29 (LMU1_A13)
- net FT_MEM1_A14: now also U5.AH27 (LMU1_A14/WE_N)
- net FT_MEM1_A15: now also U5.AG27 (LMU1_A15/CAS_N)
- net FT_MEM1_A16: now also U5.AG26 (LMU1_A16/RAS_N)
- net FT_MEM1_A17: now also U5.AP31 (LMU1_A17)
- net FT_MEM1_A2: now also U5.AH25 (LMU1_A2)
- net FT_MEM1_A3: now also U5.AP25 (LMU1_A3)
- net FT_MEM1_A4: now also U5.AN25 (LMU1_A4)
- net FT_MEM1_A5: now also U5.AM25 (LMU1_A5)
- net FT_MEM1_A6: now also U5.AJ23 (LMU1_A6)
- net FT_MEM1_A7: now also U5.AL24 (LMU1_A7)
- net FT_MEM1_A8: now also U5.AM24 (LMU1_A8)
- net FT_MEM1_A9: now also U5.AP23 (LMU1_A9)
- net FT_MEM1_ACT_N: now also U5.AJ22 (LMU1_ACT_N)
- net FT_MEM1_ALERT_N: now also U5.AH22 (LMU1_BP_ALERT_N)
- net FT_MEM1_BA0: now also U5.AH26 (LMU1_BA0)
- net FT_MEM1_BA1: now also U5.AM28 (LMU1_BA1)
- net FT_MEM1_BG0: now also U5.AK23 (LMU1_BG0)
- net FT_MEM1_BG1: now also U5.AK22 (LMU1_BG1)
- net FT_MEM1_C0: now also U5.AL30 (LMU1_C0)
- net FT_MEM1_C1: now also U5.AM31 (VSS)
- net FT_MEM1_C2: now also U5.AN32 (VSS)
- net FT_MEM1_CKE0: now also U5.AN22 (LMU1_CKE0)
- net FT_MEM1_CKE1: now also U5.AL22 (LMU1_CKE1)
- net FT_MEM1_CLK0_C: now also U5.AK25 (LMU1_CLK_C0)
- net FT_MEM1_CLK0_T: now also U5.AL25 (LMU1_CLK_T0)
- net FT_MEM1_CLK1_C: now also U5.AJ26 (LMU1_CLK_C1)
- net FT_MEM1_CLK1_T: now also U5.AK26 (LMU1_CLK_T1)
- net FT_MEM1_CS_N0: now also U5.AK28 (LMU1_CS0)
- net FT_MEM1_CS_N1: now also U5.AN31 (LMU1_CS1)
- net FT_MEM1_DQ0: now also U5.AD32 (LMU1_DQ0)
- net FT_MEM1_DQ1: now also U5.AD34 (LMU1_DQ1)
- net FT_MEM1_DQ10: now also U5.V32 (LMU1_DQ10)
- net FT_MEM1_DQ11: now also U5.V31 (LMU1_DQ11)
- net FT_MEM1_DQ12: now also U5.AA34 (LMU1_DQ12)
- net FT_MEM1_DQ13: now also U5.W32 (LMU1_DQ13)
- net FT_MEM1_DQ14: now also U5.V34 (LMU1_DQ14)
- net FT_MEM1_DQ15: now also U5.AA32 (LMU1_DQ15)
- net FT_MEM1_DQ16: now also U5.AL33 (LMU1_DQ16)
- net FT_MEM1_DQ17: now also U5.AH32 (LMU1_DQ17)
- net FT_MEM1_DQ18: now also U5.AH33 (LMU1_DQ18)
- net FT_MEM1_DQ19: now also U5.AL34 (LMU1_DQ19)
- net FT_MEM1_DQ2: now also U5.AA31 (LMU1_DQ2)
- net FT_MEM1_DQ20: now also U5.AL32 (LMU1_DQ20)
- net FT_MEM1_DQ21: now also U5.AJ31 (LMU1_DQ21)
- net FT_MEM1_DQ22: now also U5.AJ33 (LMU1_DQ22)
- net FT_MEM1_DQ23: now also U5.AM33 (LMU1_DQ23)
- net FT_MEM1_DQ24: now also U5.AG30 (LMU1_DQ24)
- net FT_MEM1_DQ25: now also U5.AE31 (LMU1_DQ25)
- net FT_MEM1_DQ26: now also U5.AE32 (LMU1_DQ26)
- net FT_MEM1_DQ27: now also U5.AH34 (LMU1_DQ27)
- net FT_MEM1_DQ28: now also U5.AG29 (LMU1_DQ28)
- net FT_MEM1_DQ29: now also U5.AH30 (LMU1_DQ29)
- net FT_MEM1_DQ3: now also U5.AB32 (LMU1_DQ3)
- net FT_MEM1_DQ30: now also U5.AF33 (LMU1_DQ30)
- net FT_MEM1_DQ31: now also U5.AF31 (LMU1_DQ31)
- net FT_MEM1_DQ32: now also U5.AP14 (LMU1_DQ32)
- net FT_MEM1_DQ33: now also U5.AN17 (LMU1_DQ33)
- net FT_MEM1_DQ34: now also U5.AP17 (LMU1_DQ34)
- net FT_MEM1_DQ35: now also U5.AN14 (LMU1_DQ35)
- net FT_MEM1_DQ36: now also U5.AL14 (LMU1_DQ36)
- net FT_MEM1_DQ37: now also U5.AM17 (LMU1_DQ37)
- net FT_MEM1_DQ38: now also U5.AP16 (LMU1_DQ38)
- net FT_MEM1_DQ39: now also U5.AM14 (LMU1_DQ39)
- net FT_MEM1_DQ4: now also U5.AE34 (LMU1_DQ4)
- net FT_MEM1_DQ40: now also U5.AH16 (LMU1_DQ40)
- net FT_MEM1_DQ41: now also U5.AH17 (LMU1_DQ41)
- net FT_MEM1_DQ42: now also U5.AK21 (LMU1_DQ42)
- net FT_MEM1_DQ43: now also U5.AJ20 (LMU1_DQ43)
- net FT_MEM1_DQ44: now also U5.AJ16 (LMU1_DQ44)
- net FT_MEM1_DQ45: now also U5.AK16 (LMU1_DQ45)
- net FT_MEM1_DQ46: now also U5.AH20 (LMU1_DQ46)
- net FT_MEM1_DQ47: now also U5.AL19 (LMU1_DQ47)
- net FT_MEM1_DQ48: now also U5.AP10 (LMU1_DQ48)
- net FT_MEM1_DQ49: now also U5.AM11 (LMU1_DQ49)
- net FT_MEM1_DQ5: now also U5.AE33 (LMU1_DQ5)
- net FT_MEM1_DQ50: now also U5.AN13 (LMU1_DQ50)
- net FT_MEM1_DQ51: now also U5.AP13 (LMU1_DQ51)
- net FT_MEM1_DQ52: now also U5.AK10 (LMU1_DQ52)
- net FT_MEM1_DQ53: now also U5.AL10 (LMU1_DQ53)
- net FT_MEM1_DQ54: now also U5.AM13 (LMU1_DQ54)
- net FT_MEM1_DQ55: now also U5.AP12 (LMU1_DQ55)
- net FT_MEM1_DQ56: now also U5.AH11 (LMU1_DQ56)
- net FT_MEM1_DQ57: now also U5.AJ15 (LMU1_DQ57)
- net FT_MEM1_DQ58: now also U5.AK15 (LMU1_DQ58)
- net FT_MEM1_DQ59: now also U5.AH12 (LMU1_DQ59)
- net FT_MEM1_DQ6: now also U5.AB33 (LMU1_DQ6)
- net FT_MEM1_DQ60: now also U5.AH10 (LMU1_DQ60)
- net FT_MEM1_DQ61: now also U5.AJ10 (LMU1_DQ61)
- net FT_MEM1_DQ62: now also U5.AH13 (LMU1_DQ62)
- net FT_MEM1_DQ63: now also U5.AH14 (LMU1_DQ63)
- net FT_MEM1_DQ64: now also U5.AP18 (LMU1_CB0)
- net FT_MEM1_DQ65: now also U5.AP21 (LMU1_CB1)
- net FT_MEM1_DQ66: now also U5.AL21 (LMU1_CB2)
- net FT_MEM1_DQ67: now also U5.AN18 (LMU1_CB3)
- net FT_MEM1_DQ68: now also U5.AL17 (LMU1_CB4)
- net FT_MEM1_DQ69: now also U5.AN20 (LMU1_CB5)
- net FT_MEM1_DQ7: now also U5.AB34 (LMU1_DQ7)
- net FT_MEM1_DQ70: now also U5.AL18 (LMU1_CB6)
- net FT_MEM1_DQ71: now also U5.AP20 (LMU1_CB7)
- net FT_MEM1_DQ8: now also U5.Y33 (LMU1_DQ8)
- net FT_MEM1_DQ9: now also U5.Y34 (LMU1_DQ9)
- net FT_MEM1_DQS_C_0: now also U5.AC34 (LMU1_DQS_C0)
- net FT_MEM1_DQS_C_1: now also U5.W34 (LMU1_DQS_C1)
- net FT_MEM1_DQS_C_10: now also U5.W31 (LMU1_DQS_C10)
- net FT_MEM1_DQS_C_11: now also U5.AK32 (LMU1_DQS_C11)
- net FT_MEM1_DQS_C_12: now also U5.AG32 (LMU1_DQS_C12)
- net FT_MEM1_DQS_C_13: now also U5.AP15 (LMU1_DQS_C13)
- net FT_MEM1_DQS_C_14: now also U5.AK18 (LMU1_DQS_C14)
- net FT_MEM1_DQS_C_15: now also U5.AP11 (LMU1_DQS_C15)
- net FT_MEM1_DQS_C_16: now also U5.AK12 (LMU1_DQS_C16)
- net FT_MEM1_DQS_C_17: now also U5.AP19 (LMU1_DQS_C17)
- net FT_MEM1_DQS_C_2: now also U5.AK34 (LMU1_DQS_C2)
- net FT_MEM1_DQS_C_3: now also U5.AG34 (LMU1_DQS_C3)
- net FT_MEM1_DQS_C_4: now also U5.AL15 (LMU1_DQS_C4)
- net FT_MEM1_DQS_C_5: now also U5.AJ19 (LMU1_DQS_C5)
- net FT_MEM1_DQS_C_6: now also U5.AL11 (LMU1_DQS_C6)
- net FT_MEM1_DQS_C_7: now also U5.AK13 (LMU1_DQS_C7)
- net FT_MEM1_DQS_C_8: now also U5.AM19 (LMU1_DQS_C8)
- net FT_MEM1_DQS_C_9: now also U5.AC31 (LMU1_DQS_C9)
- net FT_MEM1_DQS_T_0: now also U5.AC33 (LMU1_DQS_T0)
- net FT_MEM1_DQS_T_1: now also U5.W33 (LMU1_DQS_T1)
- net FT_MEM1_DQS_T_10: now also U5.Y31 (LMU1_DQS_T10)
- net FT_MEM1_DQS_T_11: now also U5.AK31 (LMU1_DQS_T11)
- net FT_MEM1_DQS_T_12: now also U5.AG31 (LMU1_DQS_T12)
- net FT_MEM1_DQS_T_13: now also U5.AN15 (LMU1_DQS_T13)
- net FT_MEM1_DQS_T_14: now also U5.AJ18 (LMU1_DQS_T14)
- net FT_MEM1_DQS_T_15: now also U5.AN11 (LMU1_DQS_T15)
- net FT_MEM1_DQS_T_16: now also U5.AJ12 (LMU1_DQS_T16)
- net FT_MEM1_DQS_T_17: now also U5.AN19 (LMU1_DQS_T17)
- net FT_MEM1_DQS_T_2: now also U5.AJ34 (LMU1_DQS_T2)
- net FT_MEM1_DQS_T_3: now also U5.AF34 (LMU1_DQS_T3)
- net FT_MEM1_DQS_T_4: now also U5.AL16 (LMU1_DQS_T4)
- net FT_MEM1_DQS_T_5: now also U5.AK19 (LMU1_DQS_T5)
- net FT_MEM1_DQS_T_6: now also U5.AL12 (LMU1_DQS_T6)
- net FT_MEM1_DQS_T_7: now also U5.AL13 (LMU1_DQS_T7)
- net FT_MEM1_DQS_T_8: now also U5.AM20 (LMU1_DQS_T8)
- net FT_MEM1_DQS_T_9: now also U5.AD31 (LMU1_DQS_T9)
- net FT_MEM1_ODT0: now also U5.AH28 (LMU1_ODT0)
- net FT_MEM1_ODT1: now also U5.AJ29 (LMU1_ODT1)
- net FT_MEM1_PAR: now also U5.AP28 (LMU1_PAR)
- net FT_MEM1_RST_N: now also U5.AG22 (LMU1_BP_MEMRESET_L)
- net GND: now also U5.AJ30 (VSS), U5.F30 (VSS)
- net VREF_CA0: now also U5.N17 (NC9)
- net VREF_CA1: now also U5.AB18 (NC10)
- net at R22.2: now also U5.P16 (LMU0_BP_ZN)
- net at R23.2: now also U5.AA17 (LMU1_BP_ZN)
Other:
- note added: "DDR4 Channel 1 1DPC, SODIMM"
- note added: "DDR4 Channel 2 1DPC, SODIMM"
- moved on the sheet: C89, C90, R22, R23
