File: d2000-mitx/d2000-mitx/12_USB.kicad_sch (KiCad schematic)
At the start: 25 parts, among them J1 USB 3.1 + PD INPUT, J3 USB3_A_Stacked, J5 Conn_02x10_Top_Bottom, U10 TPS784105QWDRBRQ1, U11 TPS784105QWDRBRQ1, U12 VL805 REAR I/O, U9 VL805 REAR I/O, Y1 Crystal_GND23, Y2 Crystal_GND23

Commit message: update schem + pcb layout
Parts:
- removed J3: USB3_A_Stacked, Connector_USB:USB_A_CUI_UJ2-ADH-TH_Horizontal_Stacked, symbol Connector:USB3_A_Stacked
- added J12: USB3_A0, Connector_USB:USB_A_Receptacle_XKB_U231-091N-4BLRA00-S, symbol Connector:USB3_A
- added J13: USB3_A1, Connector_USB:USB_A_Receptacle_XKB_U231-091N-4BLRA00-S, symbol Connector:USB3_A
- added J6: 6116151-1, 6116151_1:TE_6116151-1, symbol 6116151-1:6116151-1
Connections:
- net VL805_1_PE_RX_C_P is gone; now on net FT_PEU1_X1_C_RXP0: U12.24 (PE_TXP)
- net +3V3: now also R2.1; no longer R4.1
- net +5V: now also J12.1 (VBUS), J13.1 (VBUS), J6.13 (VCC), J6.9 (VCC)
- net EXT_P0_D+: now also J12.3 (D+)
- net EXT_P0_D-: now also J12.2 (D-)
- net EXT_P0_SSRX+: now also J12.6 (SSRX+)
- net EXT_P0_SSRX-: now also J12.5 (SSRX-)
- net EXT_P0_SSTX+: now also J12.9 (SSTX+)
- net EXT_P0_SSTX-: now also J12.8 (SSTX-)
- net EXT_P1_D+: now also J13.3 (D+)
- net EXT_P1_D-: now also J13.2 (D-)
- net EXT_P1_SSRX+: now also J13.6 (SSRX+)
- net EXT_P1_SSRX-: now also J13.5 (SSRX-)
- net EXT_P1_SSTX+: now also J13.9 (SSTX+)
- net EXT_P1_SSTX-: now also J13.8 (SSTX-)
- net EXT_P2_D+: now also J6.11 (D+)
- net EXT_P2_D-: now also J6.10 (D-)
- net GND: now also J12.10 (SHIELD), J12.4 (GND), J12.7 (DRAIN), J13.10 (SHIELD), J13.4 (GND), J13.7 (DRAIN), J6.12 (GND), J6.16 (GND)
- net at R2.2: now also U9.38 (~{USBHPE4}), U9.40 (~{USBHPE3}), U9.42 (~{USBHPE2}), U9.44 (~{USBHPE1})
- net FT_PEU1_X1_RXP0: now reaches C7.1
- net FT_PEU1_X1_C_RXP0: now reaches C7.2
- net VL805_0_PE_CLK_N renamed FT_PEU0_VL805_CLK_N
- net VL805_0_PE_CLK_P renamed FT_PEU0_VL805_CLK_P
- net VL805_1_PE_RX_C_N renamed FT_PEU1_X1_C_RXN0
- net VL805_1_PE_RX_N renamed FT_PEU1_X1_RXN0
- net VL805_1_PE_TX_N renamed FT_PEU1_X1_TXN0
- net VL805_1_PE_TX_P renamed FT_PEU1_X1_TXP0
- new net 3V3: R4.1
- new net EXT_P3_D+: J6.15 (D+)
- new net EXT_P3_D-: J6.14 (D-)
Other:
- note added: "2 USB-A 2.0 Rear"
- note added: "2 USB-A 3.0 Rear"
- note added: "2x USB-A 3.0 2x USB-A 2.0 Internal header"
- note added: "USB 3.0 Controller VL805 1 Internal I/O"
- note added: "USB 3.0 Controller VL805 1 Rear I/O"
- note added: "USB-C USB 3.1 + 20V PD Input"
- moved on the sheet: C1, C10, C11, C12, C2, C3, C4, C5, C6, C7, C8, C9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
