File: d2000-mitx/d2000-mitx/16_vdd_core.kicad_sch (KiCad schematic)
At the start: 0 parts

Commit message: update schem + pcb layout
Parts:
- added C215, C244: 1uF, Capacitor_SMD:C_0402_1005Metric, symbol Device:C_Small
- added C216, C243: 100pF, Capacitor_SMD:C_0402_1005Metric, symbol Device:C_Small
- added C217, C218, C219, C237, C238, C241: 22uF, Capacitor_SMD:C_0603_1608Metric, symbol Device:C_Small
- added C220, C221, C239, C240: 4.7uF, Capacitor_SMD:C_0603_1608Metric, symbol Device:C_Small
- added C222, C230, C231, C242, C253, C255: 0.1uF, Capacitor_SMD:C_0603_1608Metric, symbol Device:C_Small
- added C223, C245: 0.22uF, Capacitor_SMD:C_0603_1608Metric, symbol Device:C_Small
- added C224, C225, C226, C227, C246, C247, C248, C249: 47uF, Capacitor_SMD:C_1206_3216Metric, symbol Device:C_Small
- added C228, C229, C250, C252: 10uF, Capacitor_SMD:C_0603_1608Metric, symbol Device:C_Small
- added C232, C233, C234: 560uF, Capacitor_SMD:CP_Elec_6.3x5.9, symbol Device:C_Polarized_Small
- added C235: 2.2nF, Capacitor_SMD:C_0603_1608Metric, symbol Device:C_Small
- added C236: 10nF (NC), Capacitor_SMD:C_0603_1608Metric, symbol Device:C_Small
- added D1: LIFE_LED, LED_SMD:LED_0603_1608Metric, symbol Device:LED
- added L1, L2: 0.22uH, Inductor_SMD:L_APV_APH1050, symbol Device:L
- added Q2: 2N7002, Package_TO_SOT_SMD:SOT-23, symbol Transistor_FET:2N7002
- added R51: 0.01r, Resistor_SMD:R_0402_1005Metric, symbol Device:R_Small
- added R60, R61, R65, R70, R72, R73, R76, R80, R81, R82: 0r, Resistor_SMD:R_0402_1005Metric, symbol Device:R_Small
- added R62, R77: 0r (NC), Resistor_SMD:R_0402_1005Metric, symbol Device:R_Small
- added R63, R78: 2.2r, Resistor_SMD:R_0603_1608Metric, symbol Device:R_Small
- added R64, R79: 60.4k, Resistor_SMD:R_0603_1608Metric, symbol Device:R_Small
- added R66: 100k, Resistor_SMD:R_0402_1005Metric, symbol Device:R_Small
- added R67, R68, R69, R74, R86, R87, R88: 10k, Resistor_SMD:R_0402_1005Metric, symbol Device:R_Small
- added R71, R84: 30.1k, Resistor_SMD:R_0402_1005Metric, symbol Device:R_Small
- added R75: 4.7k, Resistor_SMD:R_0402_1005Metric, symbol Device:R_Small
- added R83: 680r, Resistor_SMD:R_0603_1608Metric, symbol Device:R_Small
- added R85: 560r, Resistor_SMD:R_0603_1608Metric, symbol Device:R_Small
- added TP15, TP4: VDD_CORE, symbol Connector:TestPoint
- added TP16, TP5, TP6, TP9: GND, symbol Connector:TestPoint
- added TP7, TP8: VCORE, symbol Connector:TestPoint
- added U15: MP8796GVT-P-2, TQFN-25_MP8796_MNP, symbol MP8796GVT_P:MP8796GVT-P
- added U3: MP8796GVT-P-1, TQFN-25_MP8796_MNP, symbol MP8796GVT_P:MP8796GVT-P
Connections:
- new net: R79.2, U15.20 (ILIM)
- new net: D1.1 (K), Q2.3 (D)
- new net: D1.2 (A), R83.2
- new net: C242.2, U15.18 (SS)
- new net: R80.2, U15.9 (EN)
- new net: C239.2, R78.2, U15.5 (VDRV)
- new net: R81.1, U15.10 (PG)
- new net: R84.1, U15.17 (FREQ)
- new net: C245.2, L2.1, U15.2 (SW), U15.3 (SW)
- new net: C240.2, R77.2, R78.1, U15.24 (VCC)
- new net: C245.1, U15.25 (BST)
- new net: C221.2, R62.2, R63.1, U3.24 (VCC)
- new net: C235.2, C236.2, R73.1, R75.2
- new net: C220.2, R63.2, U3.5 (VDRV)
- new net: R61.1, U3.10 (PG)
- new net: R71.1, U3.17 (FREQ)
- new net: R64.2, U3.20 (ILIM)
- new net: C223.2, L1.1, U3.2 (SW), U3.3 (SW)
- new net: C222.2, U3.18 (SS)
- new net: C223.1, U3.25 (BST)
- new net: Q2.1 (G), R85.2
- new net: R65.2, U3.13 (SET)
- new net: R60.2, U3.9 (EN)
- new net 12V: R51.1
- new net 12V_CORE: C215.2, C216.2, C217.2, C218.2, C219.2, C237.2, C238.2, C241.2, C243.2, C244.2, R51.2, U15.1 (IN), U15.16 (IN), U3.1 (IN), U3.16 (IN)
- new net 3V3: R62.1, R77.1
- new net 3v3: R83.1
- new net GND: C215.1, C216.1, C217.1, C218.1, C219.1, C220.1, C221.1, C222.1, C224.1, C225.1, C226.1, C227.1, C228.1, C229.1, C230.1, C231.1, C232.2, C233.2, C234.2, C237.1, C238.1, C239.1, C240.1, C241.1, C242.1, C243.1, C244.1, C246.1, C247.1, C248.1, C249.1, C250.1, C252.1, C253.1, C255.1, Q2.2 (S), R64.1, R71.2, R72.2, R79.1, R84.2, TP16.1, TP5.1, U15.14 (PGND), U15.15 (PGND), U15.23 (AGND), U15.4 (PGND), U3.14 (PGND), U3.15 (PGND), U3.23 (AGND), U3.4 (PGND)
- new net ISUM_M1: R70.1, U3.19 (ISUM)
- new net ISUM_M2: R70.2, U15.19 (ISUM)
- new net MODE_M1: R67.2, R86.2, U15.8 (MODE), U3.8 (MODE)
- new net PASS_M1: R76.2, U3.11 (PASS)
- new net PASS_M2: R82.2, U15.11 (PASS)
- new net PMODE_M1: R68.2, R87.2, U15.7 (PMODE), U3.7 (PMODE)
- new net RAMP_M1: R69.2, R88.2, U15.6 (RAMP), U3.6 (RAMP)
- new net RGND: C236.1, R72.1, R74.1, U15.21 (RGND), U3.21 (RGND)
- new net SET: R65.1
- new net TAKE_M1: R66.1, R82.1, U3.12 (TAKE)
- new net TAKE_M2: R76.1, U15.12 (TAKE)
- new net VCORE: C224.2, C225.2, C226.2, C227.2, C228.2, C229.2, C230.2, C231.2, C232.1, C233.1, C234.1, C246.2, C247.2, C248.2, C249.2, C250.2, C252.2, C253.2, C255.2, L1.2, L2.2, R73.2, TP15.1, TP4.1, TP6.1, TP7.1, TP8.1, TP9.1
- new net VC_FB: C235.1, R74.2, R75.1, U15.22 (FB), U3.22 (FB)
- new net VC_VCC: R66.2, R67.1, R68.1, R69.1, R86.1, R87.1, R88.1
- new net VDD_CORE_EN: R60.1, R80.1
- new net VDD_CORE_PWRGD: R61.2, R81.2, R85.1
- no-connect marks 0 -> 1
Other:
- note added: "Ilim Ilim(A)=1.8(V)/0.0604(mΩ) =29.8A"
- note added: "SW Freq = 24/30.1 (kΩ) SW Freq = 800KHz"
- note added: "Soft Start Tss(ms)=30*Css(uF) Tss=3ms"
- note added: "VDD_CORE 0.88v @ 29.8A First phase"
- note added: "VDD_CORE 0.88v @ 29.8A Second phase"
- note added: "Vout=0.6*(1+R1/R2) =0.6*(1+4.7/10) =0.882V"
