File: d2000-mitx/d2000-mitx/17_vddq.kicad_sch (KiCad schematic)
At the start: 0 parts

Commit message: update schem + pcb layout
Parts:
- added C261: 1uF, Capacitor_SMD:C_0402_1005Metric, symbol Device:C_Small
- added C262, C263, C264, C267, C268, C269, C270, C271, C272: 22uF, Capacitor_SMD:C_0603_1608Metric, symbol Device:C_Small
- added C265, C273: 0.22uF, Capacitor_SMD:C_0402_1005Metric, symbol Device:C_Small
- added C266: 560uF, Capacitor_SMD:C_1206_3216Metric, symbol Device:C_Small
- added C274, C275, C276, C277: 47uF, Capacitor_SMD:C_1206_3216Metric, symbol Device:C_Small
- added C278, C279, C280, C281: 10uF, Capacitor_SMD:C_0603_1608Metric, symbol Device:C_Small
- added D4: LED, symbol Device:LED
- added L4: 0.68uH, symbol Device:L
- added NB687: ~, symbol NB687GQ:NB687GQ
- added Q3: 2N7002, Package_TO_SOT_SMD:SOT-23, symbol Transistor_FET:2N7002
- added R100, R101: 10k, Resistor_SMD:R_0402_1005Metric, symbol Device:R_Small
- added R102, R103: 560r, Resistor_SMD:R_0402_1005Metric, symbol Device:R_Small
- added R94: 0r, Resistor_SMD:R_0402_1005Metric, symbol Device:R_Small
- added R95, R96, R97: 100k, Resistor_SMD:R_0402_1005Metric, symbol Device:R_Small
- added R98: 5.11r, Resistor_SMD:R_0402_1005Metric, symbol Device:R_Small
- added R99: 0.01r, Resistor_SMD:R_1206_3216Metric, symbol Device:R_Small
- added TP10: VDDQ, symbol Connector:TestPoint
- added TP11: VDDQ_PWRGD, symbol Connector:TestPoint
- added TP12: PWR_S3, symbol Connector:TestPoint
- added TP13: PWR_S5, symbol Connector:TestPoint
- added TP14: VREF_CA0, symbol Connector:TestPoint
Connections:
- new net: Q3.1 (G), R103.1
- new net: D4.1 (K), Q3.3 (D)
- new net: C261.2, NB687.3 (3V3), R98.2
- new net: NB687.13 (FB), R100.1, R101.2
- new net: C265.1, NB687.9 (SW)
- new net: C265.2, L4.1, NB687.10 (BST)
- new net: C262.2, C263.2, NB687.1 (VIN), R99.2
- new net: NB687.14 (MODE), R94.2
- new net: C273.2, NB687.7 (VTTREF)
- new net: D4.2 (A), R102.1
- new net 3V3: R95.2, R98.1
- new net 3V3_S3: C264.1, NB687.8 (VPPIN), R102.2
- new net 5V_S3: R99.1
- new net GND: C261.1, C262.1, C263.1, C264.2, C266.1, C267.1, C268.1, C269.1, C270.1, C271.1, C272.1, C274.1, C275.1, C276.1, C277.1, C278.1, C279.1, C280.1, C281.1, NB687.2 (PGND), NB687.4 (AGND), Q3.2 (S), R101.1, R94.1, R96.2, R97.2
- new net PWR_S3: NB687.16 (EN1), R97.1, TP12.1
- new net PWR_S5: NB687.15 (EN2), R96.1, TP13.1
- new net VDDQ: C266.2, C267.2, C268.2, C274.2, C275.2, C276.2, C277.2, C278.2, C279.2, C280.2, C281.2, L4.2, NB687.6 (VDDQ), R100.2, TP10.1
- new net VDDQ_PWRGD: NB687.12 (PG), R103.2, R95.1, TP11.1
- new net VPP: C271.2, C272.2, NB687.11 (VPP)
- new net VREF_CA0: C273.1, TP14.1
- new net VTT: C269.2, C270.2, NB687.5 (VTT)
Other:
- note added: "MPS NB687 1.2V 8A VDDQ Buck"
- note added: "Testpoints"
