File: d2000-mitx/d2000-mitx/02_power_block.kicad_sch (KiCad schematic)
At the start: 0 parts

Commit message: update schem + pcb layout
Other:
- note added: "+0.6V"
- note added: "+0.88V"
- note added: "+1.05V"
- note added: "+1.2V"
- note added: "+1.8V"
- note added: "+12V"
- note added: "+2.5V"
- note added: "+3.3V"
- note added: "+5V"
- note added: "ALC662"
- note added: "AP2112K-1.8"
- note added: "AP61300Z6-7"
- note added: "ATX Mode"
- note added: "ATX POWER"
- note added: "Bead"
- note added: "D2000"
- note added: "DIMM DDR4"
- note added: "Device"
- note added: "EC (RP2354)"
- note added: "FAN"
- note added: "M.2_1"
- note added: "MOS AO4606"
- note added: "MP8796 x2"
- note added: "NB687"
- note added: "NMOS"
- note added: "OFF"
- note added: "ON"
- note added: "P12V"
- note added: "P1V05"
- note added: "P1V8_STBY"
- note added: "P3V3"
- note added: "P3V3_S3"
- note added: "P3V3_STBY"
- note added: "P5V"
- note added: "P5V_S3"
- note added: "PCIE SLOT"
- note added: "PEU_AVDD/AVDDCLK"
- note added: "RTC (fill)"
- note added: "S0"
- note added: "S3"
- note added: "S4 & 5"
- note added: "SI52147"
- note added: "USB3.0*4"
- note added: "VCORE"
- note added: "VDDQ"
- note added: "VDD_IO"
- note added: "VL805"
- note added: "VPP"
- note added: "VTT"
