File: d2000-mitx/d2000-mitx/09_pcie.kicad_sch (KiCad schematic)
At the start: 3 parts, among them CN1 2EG08217-D2D-DF, J4 M.2_NVME, J6 M.2_WIFI

Commit message: update schem + pcb layout
Parts:
- removed J6: M.2_WIFI, 2199119-3-M.2:CONN75_2199119-3_TEC, symbol Connector:Bus_M.2_Socket_E
- added C195, C196, C206, C207, C208, C209, C210, C93, C94: 0.1uF, Capacitor_SMD:C_0402_1005Metric, symbol Device:C_Small
- added C197, C200: 4.7uF, Capacitor_SMD:C_0603_1608Metric, symbol Device:C_Small
- added C198, C199: 270uF, Capacitor_Tantalum_SMD:CP_EIA-7361-38_AVX-V, symbol Device:C_Polarized
- added C201, C202, C203, C204: 0.1uF, Capacitor_SMD:C_0603_1608Metric, symbol Device:C_Small
- added C205: 4.7uF, Capacitor_SMD:C_1206_3216Metric, symbol Device:C_Small
- added FB1, FB2: 100M, 120r, 2A, symbol Device:FerriteBead_Small
- added J11: M.2_NVME1, m.2-m1_2199119_5:TE_1-2199119-5, symbol Connector:Bus_M.2_Socket_M
- added R52, R53, R54, R59: 4.7k, Resistor_SMD:R_0402_1005Metric, symbol Device:R_Small
- added R55, R56, R57, R58: 0r, Resistor_SMD:R_0402_1005Metric, symbol Device:R_Small
- J4: value M.2_NVME -> M.2_NVME0; footprint 2199119-3-M.2:CONN75_2199119-3_TEC -> m.2-m1_2199119_5:TE_1-2199119-5
Connections:
- net FT_PEU0_RXN0: now also J11.41 (PERn0/SATA-B+); no longer CN1.A17 (PERN0)
- net FT_PEU0_RXN1: now also J11.29 (PERn1); no longer CN1.A22 (PERN1)
- net FT_PEU0_RXN10: now also J4.17 (PERn2); no longer CN1.A61 (PERN10)
- net FT_PEU0_RXN11: now also J4.5 (PERn3); no longer CN1.A65 (PERN11)
- net FT_PEU0_RXN12: no longer CN1.A69 (PERN12)
- net FT_PEU0_RXN13: no longer CN1.A73 (PERN13)
- net FT_PEU0_RXN14: no longer CN1.A77 (PERN14)
- net FT_PEU0_RXN15: no longer CN1.A81 (PERN15)
- net FT_PEU0_RXN2: now also J11.17 (PERn2); no longer CN1.A26 (PERN2)
- net FT_PEU0_RXN3: now also J11.5 (PERn3); no longer CN1.A30 (PERN3)
- net FT_PEU0_RXN8: now also J4.41 (PERn0/SATA-B+); no longer CN1.A53 (PERN8)
- net FT_PEU0_RXN9: now also J4.29 (PERn1); no longer CN1.A57 (PERN9)
- net FT_PEU0_RXP0: now also J11.43 (PERp0/SATA-B-); no longer CN1.A16 (PERP0)
- net FT_PEU0_RXP1: now also J11.31 (PERp1); no longer CN1.A21 (PERP1)
- net FT_PEU0_RXP10: now also J4.19 (PERp2); no longer CN1.A60 (PERP10)
- net FT_PEU0_RXP11: now also J4.7 (PERp3); no longer CN1.A64 (PERP11)
- net FT_PEU0_RXP12: no longer CN1.A68 (PERP12)
- net FT_PEU0_RXP13: no longer CN1.A72 (PERP13)
- net FT_PEU0_RXP14: no longer CN1.A76 (PERP14)
- net FT_PEU0_RXP15: no longer CN1.A80 (PERP15)
- net FT_PEU0_RXP2: now also J11.19 (PERp2); no longer CN1.A25 (PERP2)
- net FT_PEU0_RXP3: now also J11.7 (PERp3); no longer CN1.A29 (PERP3)
- net FT_PEU0_RXP8: now also J4.43 (PERp0/SATA-B-); no longer CN1.A52 (PERP8)
- net FT_PEU0_RXP9: now also J4.31 (PERp1); no longer CN1.A56 (PERP9)
- net FT_PEU0_TXN0: now also J11.47 (PETn0/SATA-A-); no longer CN1.B15 (PETN0)
- net FT_PEU0_TXN1: now also J11.35 (PETn1); no longer CN1.B20 (PETN1)
- net FT_PEU0_TXN10: now also J4.23 (PETn2); no longer CN1.B59 (PETN10)
- net FT_PEU0_TXN11: now also J4.11 (PETn3); no longer CN1.B63 (PETN11)
- net FT_PEU0_TXN12: no longer CN1.B67 (PETN12)
- net FT_PEU0_TXN13: no longer CN1.B71 (PETN13)
- net FT_PEU0_TXN14: no longer CN1.B75 (PETN14)
- net FT_PEU0_TXN15: no longer CN1.B79 (PETN15)
- net FT_PEU0_TXN2: now also J11.23 (PETn2); no longer CN1.B24 (PETN2)
- net FT_PEU0_TXN3: now also J11.11 (PETn3); no longer CN1.B28 (PETN3)
- net FT_PEU0_TXN8: now also J4.47 (PETn0/SATA-A-); no longer CN1.B51 (PETN8)
- net FT_PEU0_TXN9: now also J4.35 (PETn1); no longer CN1.B55 (PETN9)
- net FT_PEU0_TXP0: now also J11.49 (PETp0/SATA-A+); no longer CN1.B14 (PETP0)
- net FT_PEU0_TXP1: now also J11.37 (PETp1); no longer CN1.B19 (PETP1)
- net FT_PEU0_TXP10: now also J4.25 (PETp2); no longer CN1.B58 (PETP10)
- net FT_PEU0_TXP11: now also J4.13 (PETp3); no longer CN1.B62 (PETP11)
- net FT_PEU0_TXP12: no longer CN1.B66 (PETP12)
- net FT_PEU0_TXP13: no longer CN1.B70 (PETP13)
- net FT_PEU0_TXP14: no longer CN1.B74 (PETP14)
- net FT_PEU0_TXP15: no longer CN1.B78 (PETP15)
- net FT_PEU0_TXP2: now also J11.25 (PETp2); no longer CN1.B23 (PETP2)
- net FT_PEU0_TXP3: now also J11.13 (PETp3); no longer CN1.B27 (PETP3)
- net FT_PEU0_TXP8: now also J4.49 (PETp0/SATA-A+); no longer CN1.B50 (PETP8)
- net FT_PEU0_TXP9: now also J4.37 (PETp1); no longer CN1.B54 (PETP9)
- net FT_PEU1_RXN0: now also CN1.A17 (PERN0); no longer J4.41 (PERn0/SATA-B+)
- net FT_PEU1_RXN1: now also CN1.A22 (PERN1); no longer J4.29 (PERn1)
- net FT_PEU1_RXN2: now also CN1.A26 (PERN2); no longer J4.17 (PERn2)
- net FT_PEU1_RXN3: now also CN1.A30 (PERN3); no longer J4.5 (PERn3)
- net FT_PEU1_RXN8: now also CN1.A53 (PERN8)
- net FT_PEU1_RXN9: now also CN1.A57 (PERN9)
- net FT_PEU1_RXP0: now also CN1.A16 (PERP0); no longer J4.43 (PERp0/SATA-B-)
- net FT_PEU1_RXP1: now also CN1.A21 (PERP1); no longer J4.31 (PERp1)
- net FT_PEU1_RXP2: now also CN1.A25 (PERP2); no longer J4.19 (PERp2)
- net FT_PEU1_RXP3: now also CN1.A29 (PERP3); no longer J4.7 (PERp3)
- net FT_PEU1_RXP8: now also CN1.A52 (PERP8)
- net FT_PEU1_RXP9: now also CN1.A56 (PERP9)
- net FT_PEU1_TXN0: now also CN1.B15 (PETN0); no longer J4.47 (PETn0/SATA-A-)
- net FT_PEU1_TXN1: now also CN1.B20 (PETN1); no longer J4.35 (PETn1)
- net FT_PEU1_TXN2: now also CN1.B24 (PETN2); no longer J4.23 (PETn2)
- net FT_PEU1_TXN3: now also CN1.B28 (PETN3); no longer J4.11 (PETn3)
- net FT_PEU1_TXN8: now also CN1.B51 (PETN8)
- net FT_PEU1_TXN9: now also CN1.B55 (PETN9)
- net FT_PEU1_TXP0: now also CN1.B14 (PETP0); no longer J4.49 (PETp0/SATA-A+)
- net FT_PEU1_TXP1: now also CN1.B19 (PETP1); no longer J4.37 (PETp1)
- net FT_PEU1_TXP2: now also CN1.B23 (PETP2); no longer J4.25 (PETp2)
- net FT_PEU1_TXP3: now also CN1.B27 (PETP3); no longer J4.13 (PETp3)
- net FT_PEU1_TXP8: now also CN1.B50 (PETP8)
- net FT_PEU1_TXP9: now also CN1.B54 (PETP9)
- net GND: now reaches J4.1 (GND), J4.15 (GND), J4.21 (GND), J4.27 (GND), J4.3 (GND), J4.33 (GND), J4.39 (GND), J4.45 (GND), J4.51 (GND), J4.57 (GND), J4.71 (GND), J4.73 (GND), J4.75 (GND), J4.9 (GND)
- net GND: now also CN1.A1 (PRSNT1#), CN1.A12 (GND), CN1.A15 (GND), CN1.A18 (GND), CN1.A20 (GND), CN1.A23 (GND), CN1.A24 (GND), CN1.A27 (GND), CN1.A28 (GND), CN1.A31 (GND), CN1.A34 (GND), CN1.A37 (GND), CN1.A38 (GND), CN1.A4 (GND), CN1.A41 (GND), CN1.A42 (GND), CN1.A45 (GND), CN1.A46 (GND), CN1.A49 (GND), CN1.A51 (GND), CN1.A54 (GND), CN1.A55 (GND), CN1.A58 (GND), CN1.A59 (GND), CN1.A62 (GND), CN1.A63 (GND), CN1.A66 (GND), CN1.A67 (GND), CN1.A70 (GND), CN1.A71 (GND), CN1.A74 (GND), CN1.A75 (GND), CN1.A78 (GND), CN1.A79 (GND), CN1.A82 (GND), CN1.B13 (GND), CN1.B16 (GND), CN1.B18 (GND), CN1.B21 (GND), CN1.B22 (GND), CN1.B25 (GND), CN1.B26 (GND), CN1.B29 (GND), CN1.B32 (GND), CN1.B35 (GND), CN1.B36 (GND), CN1.B39 (GND), CN1.B4 (GND), CN1.B40 (GND), CN1.B43 (GND), CN1.B44 (GND), CN1.B47 (GND), CN1.B49 (GND), CN1.B52 (GND), CN1.B53 (GND), CN1.B56 (GND), CN1.B57 (GND), CN1.B60 (GND), CN1.B61 (GND), CN1.B64 (GND), CN1.B65 (GND), CN1.B68 (GND), CN1.B69 (GND), CN1.B7 (GND), CN1.B72 (GND), CN1.B73 (GND), CN1.B76 (GND), CN1.B77 (GND), CN1.B80 (GND), CN1.B82 (GND), C197.2, C198.2, C199.2, C200.2, J11.1 (GND), J11.15 (GND), J11.21 (GND), J11.27 (GND), J11.3 (GND), J11.33 (GND), J11.39 (GND), J11.45 (GND), J11.51 (GND), J11.57 (GND), J11.71 (GND), J11.73 (GND), J11.75 (GND), J11.9 (GND)
- net M2_LED0: now reaches J4.10 (DAS/~{DSS}/~{LED1})
- net 3V3: now reaches J4.12 (3.3V), J4.14 (3.3V), J4.16 (3.3V), J4.18 (3.3V), J4.2 (3.3V), J4.4 (3.3V), J4.70 (3.3V), J4.72 (3.3V), J4.74 (3.3V)
- net 3V3: now also CN1.A10 (3V3), CN1.A9 (3V3), CN1.B8 (3V3), FB1.1, FB2.1, J11.12 (3.3V), J11.14 (3.3V), J11.16 (3.3V), J11.18 (3.3V), J11.2 (3.3V), J11.4 (3.3V), J11.70 (3.3V), J11.72 (3.3V), J11.74 (3.3V), R53.1, R54.1
- net FT_PCIE_NVME_RST: now reaches J4.50 (~{PERST})
- net FT_PCIE_NVME_RST: now also J11.50 (~{PERST})
- net at J4.53 (REFCLKn): now also C204.2
- net at J4.55 (REFCLKp): now also C203.2
- net FT_PCIE_SLOT0_RST: now reaches CN1.A11 (PERST#)
- net FT_PCIE_SLOT0_RST: now also R56.1
- net FT_PCIE_SLOT0_CLKP: now reaches CN1.A13 (REFCLK+)
- net FT_PCIE_SLOT0_CLKN: now reaches CN1.A14 (REFCLK-)
- net PCIE_12V: now reaches CN1.A2 (12V)
- net PCIE_12V: now also CN1.A3 (12V), CN1.B1 (12V), CN1.B2 (12V), CN1.B3 (12V), C197.1, C198.1
- net 3V3_STANDBY: now reaches CN1.B10 (3V3_AUX)
- net 3V3_STANDBY: now also R52.1
- net at CN1.B11 (WAKE#): now also R52.2, R55.2
- net at CN1.B5 (SMCLK): now also R54.2
- net at CN1.B6 (SMDAT): now also R53.2
- net FT_PEU0_RXN4 renamed FT_PEU1_RXN4
- net FT_PEU0_RXN5 renamed FT_PEU1_RXN5
- net FT_PEU0_RXN6 renamed FT_PEU1_RXN6
- net FT_PEU0_RXN7 renamed FT_PEU1_RXN7
- net FT_PEU0_RXP4 renamed FT_PEU1_RXP4
- net FT_PEU0_RXP5 renamed FT_PEU1_RXP5
- net FT_PEU0_RXP6 renamed FT_PEU1_RXP6
- net FT_PEU0_RXP7 renamed FT_PEU1_RXP7
- net FT_PEU0_TXN4 renamed FT_PEU1_TXN4
- net FT_PEU0_TXN5 renamed FT_PEU1_TXN5
- net FT_PEU0_TXN6 renamed FT_PEU1_TXN6
- net FT_PEU0_TXN7 renamed FT_PEU1_TXN7
- net FT_PEU0_TXP4 renamed FT_PEU1_TXP4
- net FT_PEU0_TXP5 renamed FT_PEU1_TXP5
- net FT_PEU0_TXP6 renamed FT_PEU1_TXP6
- net FT_PEU0_TXP7 renamed FT_PEU1_TXP7
- new net: C195.2, C196.2, C205.2, C206.2, C207.2, C208.2, C209.2, C210.2, C93.2, C94.2
- new net: C202.2, J11.53 (REFCLKn)
- new net: C201.2, J11.55 (REFCLKp)
- new net FT_PCIE_SLOT1_RST: R57.1
- new net FT_PCIE_SLOT2_RST: R58.1
- new net FT_PEU1_RXN10: CN1.A61 (PERN10)
- new net FT_PEU1_RXN11: CN1.A65 (PERN11)
- new net FT_PEU1_RXN12: CN1.A69 (PERN12)
- new net FT_PEU1_RXN13: CN1.A73 (PERN13)
- new net FT_PEU1_RXN14: CN1.A77 (PERN14)
- new net FT_PEU1_RXN15: CN1.A81 (PERN15)
- new net FT_PEU1_RXP10: CN1.A60 (PERP10)
- new net FT_PEU1_RXP11: CN1.A64 (PERP11)
- new net FT_PEU1_RXP12: CN1.A68 (PERP12)
- new net FT_PEU1_RXP13: CN1.A72 (PERP13)
- new net FT_PEU1_RXP14: CN1.A76 (PERP14)
- new net FT_PEU1_RXP15: CN1.A80 (PERP15)
- new net FT_PEU1_TXN10: CN1.B59 (PETN10)
- new net FT_PEU1_TXN11: CN1.B63 (PETN11)
- new net FT_PEU1_TXN12: CN1.B67 (PETN12)
- new net FT_PEU1_TXN13: CN1.B71 (PETN13)
- new net FT_PEU1_TXN14: CN1.B75 (PETN14)
- new net FT_PEU1_TXN15: CN1.B79 (PETN15)
- new net FT_PEU1_TXP10: CN1.B58 (PETP10)
- new net FT_PEU1_TXP11: CN1.B62 (PETP11)
- new net FT_PEU1_TXP12: CN1.B66 (PETP12)
- new net FT_PEU1_TXP13: CN1.B70 (PETP13)
- new net FT_PEU1_TXP14: CN1.B74 (PETP14)
- new net FT_PEU1_TXP15: CN1.B78 (PETP15)
- new net M2_LED1: J11.10 (DAS/~{DSS}/~{LED1})
- new net PCIE_3V3: C195.1, C196.1, C199.1, C200.1, C205.1, C206.1, C207.1, C208.1, C209.1, C210.1, C93.1, C94.1, FB1.2, FB2.2
- new net PCIE_3V3_STANDBY: R59.1
- new net PCIE_NVME_CLKN: C202.1, C204.1
- new net PCIE_NVME_CLKP: C201.1, C203.1
- new net PCIE_RST_N: R56.2, R57.2, R58.2, R59.2
- new net PCIE_WAKE#: R55.1
Other:
- note added: "M.2 M-Key Shorter port"
- note added: "M.2 M-Key Taller port"
- note added: "PCIe 3.0 16x"
- note added: "PCIe slots"

Commit message: update schem + pcb layout
Parts:
- added C260, C282: 18pF, Capacitor_SMD:C_0402_1005Metric, symbol Device:C_Small
- added C283, C284, C285, C286, C287, C288, C289, C290, C291, C292, C293, C294, C295, C296, C297: 0.1uF, Capacitor_SMD:C_0402_1005Metric, symbol Device:C_Small
- added FB3, FB4: 100M 120R, symbol Device:FerriteBead_Small
- added R109, R110, R111, R112, R113, R114, R115, R116, R117, R118: 4.7k, Resistor_SMD:R_0402_1005Metric, symbol Device:R_Small
- added U2: SI52147-A01AGM, SI52147_A01AGM:QFN15.75P236X236X100-48_SKY-L, symbol SI52147_A01AGM:SI52147-A01AGM
- added Y4: Crystal_GND24, symbol Device:Crystal_GND24
Connections:
- net 3V3: now also C287.2, C290.2, C291.2, C292.2, C293.2, C294.2, C295.2, C296.2, C297.2, FB3.1; no longer CN1.A10 (3V3), CN1.A9 (3V3), CN1.B8 (3V3), R53.1, R54.1
- net FT_PCIE_SLOT0_CLKN: now also U2.15 (*DIFF0)
- net FT_PCIE_SLOT0_CLKP: now also U2.14 (DIFF0)
- net GND: now also C260.2, C282.1, C283.1, C284.1, C285.1, C286.1, C287.1, C288.1, C289.1, C290.1, C291.1, C292.1, C293.1, C294.1, C295.1, C296.1, C297.1, Y4.2, Y4.4
- net PCIE_3V3: now also CN1.A10 (3V3), CN1.A9 (3V3), CN1.B8 (3V3), R53.1, R54.1
- net PCIE_3V3_STANDBY renamed 3V3_STBY
- net 3V3_STBY: now also C289.2, FB4.1
- net PCIE_NVME_CLKN renamed PCIE_NVME0_CLKN
- net PCIE_NVME0_CLKN: now also U2.18 (*DIFF1); no longer C202.1
- net PCIE_NVME_CLKP renamed PCIE_NVME0_CLKP
- net PCIE_NVME0_CLKP: now also U2.17 (DIFF1); no longer C201.1
- new net: R117.1, U2.38 (SDATA)
- new net: R110.2, U2.3 (OE_DIFF0)
- new net: U2.1 (VDD_DIFF), U2.12 (VDD_DIFF), U2.13 (VDD_DIFF), U2.2 (VDD_DIFF), U2.23 (VDD_DIFF)
- new net: R113.2, U2.10 (OE_DIFF[4:5])
- new net: R114.2, U2.11 (OE_DIFF[6:8])
- new net: U2.16 (VSS_DIFF), U2.24 (VSS_DIFF), U2.6 (VSS_DIFF), U2.7 (VSS_DIFF)
- new net: U2.29 (VSS_DIFF), U2.45 (VSS_CORE), U2.46 (VSS_DIFF), U2.49 (GND)
- new net: R118.1, U2.37 (SCLK)
- new net: R116.1, U2.39 (CKPWRGD/PDB)
- new net: R109.2, U2.4 (OE_DIFF1)
- new net: U2.41 (XOUT), Y4.3
- new net: C282.2, U2.42 (XIN/CLKIN), Y4.1
- new net: R115.2, U2.5 (SSON)
- new net: R111.2, U2.8 (OE_DIFF2)
- new net: R112.2, U2.9 (OE_DIFF3)
- new net 3V3_CLK: C283.2, C284.2, C285.2, C286.2, C288.2, FB3.2, FB4.2, R109.1, R110.1, R111.1, R112.1, R113.1, R114.1, R115.1, R116.2, R117.2, R118.2, U2.34 (VDD_DIFF), U2.40 (VDD_CORE)
- new net FT_PEU0_X1_X16_CLKN: U2.30 (*DIFF6)
- new net FT_PEU0_X1_X16_CLKP: U2.31 (DIFF6)
- new net FT_PEU1_X16_CLKN: U2.32 (*DIFF7)
- new net FT_PEU1_X16_CLKP: U2.33 (DIFF7)
- new net FT_PEU1_X1_CLKN: U2.35 (*DIFF8)
- new net FT_PEU1_X1_CLKP: U2.36 (DIFF8)
- new net PCIE_NVME1_CLKN: C202.1, U2.20 (*DIFF2)
- new net PCIE_NVME1_CLKP: C201.1, U2.19 (DIFF2)
- new net PCIE_VL805_0_CLKN: U2.25 (*DIFF4)
- new net PCIE_VL805_0_CLKP: U2.26 (DIFF4)
- new net PCIE_VL805_1_CLKN: U2.27 (*DIFF5)
- new net PCIE_VL805_1_CLKP: U2.28 (DIFF5)
Other:
- note added: "PCIe Clock Generator"
- moved on the sheet: C195, C196, C197, C198, C199, C200, C203, C204, C205, C206, C207, C208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
