File: d2000-mitx/d2000-mitx/d2000-mitx.kicad_pcb (KiCad board)
At the start: 6 copper layers, 170 x 170 mm, 39 parts, among them J1 USB 3.1 + PD INPUT, J3 USB3_A_Stacked, J4 M.2_NVME, J6 M.2_WIFI, U10 TPS784105QWDRBRQ1, U11 TPS784105QWDRBRQ1, U12 VL805 REAR I/O, U13 RP2040, U4 FUSB302B01MPX, U8 W25Q32JVSS, U9 VL805 REAR I/O, Y1 Crystal_GND23, Y2 Crystal_GND23, Y3 12MHz

Commit message: added major components + updated schematic + found reference schematics to steal from
Parts:
- removed the J3 at (227.0, 24.6)
- added C100: 0.1uF, Capacitor_SMD:C_0402_1005Metric, F.Cu at (0.94, 12.3)
- added C101: 0.1uF, Capacitor_SMD:C_0402_1005Metric, F.Cu at (0.94, 14.3)
- added C102: 0.1uF, Capacitor_SMD:C_0402_1005Metric, F.Cu at (0.94, 16.2)
- added C103: 0.1uF, Capacitor_SMD:C_0402_1005Metric, F.Cu at (3.81, 0.48)
- added C104: 0.1uF, Capacitor_SMD:C_0402_1005Metric, F.Cu at (3.81, 2.46)
- added C105: 0.1uF, Capacitor_SMD:C_0402_1005Metric, F.Cu at (3.81, 4.42)
- added C106: 0.1uF, Capacitor_SMD:C_0402_1005Metric, F.Cu at (3.81, 6.39)
- added C107: 0.1uF, Capacitor_SMD:C_0402_1005Metric, F.Cu at (3.81, 8.37)
- added C108: 0.1uF, Capacitor_SMD:C_0402_1005Metric, F.Cu at (3.81, 10.3)
- added C109: 0.1uF, Capacitor_SMD:C_0402_1005Metric, F.Cu at (3.81, 12.3)
- added C110: 0.1uF, Capacitor_SMD:C_0402_1005Metric, F.Cu at (3.81, 14.3)
- added C111: 0.1uF, Capacitor_SMD:C_0402_1005Metric, F.Cu at (3.81, 16.2)
- added C112: 0.1uF, Capacitor_SMD:C_0402_1005Metric, F.Cu at (6.67, 0.48)
- added C113: 0.1uF, Capacitor_SMD:C_0402_1005Metric, F.Cu at (6.67, 2.46)
- added C114: 0.1uF, Capacitor_SMD:C_0402_1005Metric, F.Cu at (6.67, 4.42)
- added C115: 0.1uF, Capacitor_SMD:C_0402_1005Metric, F.Cu at (6.67, 6.39)
- added C116: 0.1uF, Capacitor_SMD:C_0402_1005Metric, F.Cu at (6.67, 8.37)
- added C117: 560uF, Capacitor_SMD:C_0402_1005Metric, F.Cu at (6.67, 10.3)
- added C118: 560uF, Capacitor_SMD:C_0402_1005Metric, F.Cu at (6.67, 12.3)
- added C119: 560uF, Capacitor_SMD:C_0402_1005Metric, F.Cu at (6.67, 14.3)
- added C120: 560uF, Capacitor_SMD:C_0402_1005Metric, F.Cu at (6.67, 16.2)
- added C121: 22uF, Capacitor_SMD:C_0402_1005Metric, F.Cu at (9.54, 0.48)
- added C122: 22uF, Capacitor_SMD:C_0402_1005Metric, F.Cu at (9.54, 2.46)
- added C123: 22uF, Capacitor_SMD:C_0402_1005Metric, F.Cu at (9.54, 4.42)
- added C124: 22uF, Capacitor_SMD:C_0402_1005Metric, F.Cu at (9.54, 6.39)
- added C125: 22uF, Capacitor_SMD:C_0402_1005Metric, F.Cu at (9.54, 8.37)
- added C126: 22uF, Capacitor_SMD:C_0402_1005Metric, F.Cu at (9.54, 10.3)
- added C127: 22uF, Capacitor_SMD:C_0402_1005Metric, F.Cu at (9.54, 12.3)
- added C128: 22uF, Capacitor_SMD:C_0402_1005Metric, F.Cu at (9.54, 14.3)
- added C129: 22uF, Capacitor_SMD:C_0402_1005Metric, F.Cu at (9.54, 16.2)
- added C130: 22uF, Capacitor_SMD:C_0402_1005Metric, F.Cu at (12.4, 0.48)
- added C131: 22uF, Capacitor_SMD:C_0402_1005Metric, F.Cu at (12.4, 2.46)
- added C132: 22uF, Capacitor_SMD:C_0402_1005Metric, F.Cu at (12.4, 4.42)
- added C133: 22uF, Capacitor_SMD:C_0402_1005Metric, F.Cu at (12.4, 6.39)
- added C134: 22uF, Capacitor_SMD:C_0402_1005Metric, F.Cu at (12.4, 8.37)
- added C135: 10uF, Capacitor_SMD:C_0402_1005Metric, F.Cu at (12.4, 10.3)
- added C136: 10uF, Capacitor_SMD:C_0402_1005Metric, F.Cu at (12.4, 12.3)
- added C137: 0.1uF, Capacitor_SMD:C_0402_1005Metric, F.Cu at (12.4, 14.3)
- added C138: 0.1uF, Capacitor_SMD:C_0402_1005Metric, F.Cu at (12.4, 16.2)
- added C139: 10uF, Capacitor_SMD:C_0402_1005Metric, F.Cu at (15.3, 0.48)
- added C140: 10uF, Capacitor_SMD:C_0402_1005Metric, F.Cu at (15.3, 2.46)
- added C141: 10uF, Capacitor_SMD:C_0402_1005Metric, F.Cu at (15.3, 4.42)
- added C142: 10uF, Capacitor_SMD:C_0402_1005Metric, F.Cu at (15.3, 6.39)
- added C143: 4.7uF, Capacitor_SMD:C_0402_1005Metric, F.Cu at (15.3, 8.37)
- added C144: 4.7uF, Capacitor_SMD:C_0402_1005Metric, F.Cu at (15.3, 10.3)
- added C145: 560uF, Capacitor_SMD:C_0402_1005Metric, F.Cu at (20.2, 2.46)
- added C146: 560uF, Capacitor_SMD:C_0402_1005Metric, F.Cu at (20.2, 4.42)
- added C147: 560uF, Capacitor_SMD:C_0402_1005Metric, F.Cu at (20.2, 6.39)
- added C148: 560uF, Capacitor_SMD:C_0402_1005Metric, F.Cu at (20.2, 8.37)
- added C149: 22uF, Capacitor_SMD:C_0402_1005Metric, F.Cu at (20.2, 10.3)
- added C15: 0.22uF, Capacitor_SMD:C_0402_1005Metric, F.Cu at (-8.93, 21.9)
- added C150: 0.1uF, Capacitor_SMD:C_0402_1005Metric, F.Cu at (20.2, 12.3)
- added C151: 0.1uF, Capacitor_SMD:C_0402_1005Metric, F.Cu at (20.2, 14.3)
- added C152: 10uF, Capacitor_SMD:C_0402_1005Metric, F.Cu at (20.2, 16.2)
- added C153: 22uF, Capacitor_SMD:C_0402_1005Metric, F.Cu at (23.0, 0.48)
- added C154: 0.1uF, Capacitor_SMD:C_0402_1005Metric, F.Cu at (23.0, 2.46)
- added C155: 0.1uF, Capacitor_SMD:C_0402_1005Metric, F.Cu at (23.0, 4.42)
- added C156: 10uF, Capacitor_SMD:C_0402_1005Metric, F.Cu at (23.0, 6.39)
- added C157: 22uF, Capacitor_SMD:C_0402_1005Metric, F.Cu at (23.0, 8.37)
- added C158: 0.1uF, Capacitor_SMD:C_0402_1005Metric, F.Cu at (23.0, 10.3)
- added C159: 0.1uF, Capacitor_SMD:C_0402_1005Metric, F.Cu at (23.0, 12.3)
- added C16: 0.22uF, Capacitor_SMD:C_0402_1005Metric, F.Cu at (-8.93, 23.8)
- added C160: 0.1uF, Capacitor_SMD:C_0402_1005Metric, F.Cu at (23.0, 14.3)
- added C161: 22uF, Capacitor_SMD:C_0402_1005Metric, F.Cu at (23.0, 16.2)
- added C162: 0.1uF, Capacitor_SMD:C_0402_1005Metric, F.Cu at (25.9, 0.48)
- added C163: 0.1uF, Capacitor_SMD:C_0402_1005Metric, F.Cu at (25.9, 2.46)
- added C164: 0.1uF, Capacitor_SMD:C_0402_1005Metric, F.Cu at (25.9, 4.42)
- added C165: 22uF, Capacitor_SMD:C_0402_1005Metric, F.Cu at (25.9, 6.39)
- added C166: 0.1uF, Capacitor_SMD:C_0402_1005Metric, F.Cu at (25.9, 8.37)
- added C167: 0.1uF, Capacitor_SMD:C_0402_1005Metric, F.Cu at (25.9, 10.3)
- added C168: 22uF, Capacitor_SMD:C_0402_1005Metric, F.Cu at (25.9, 12.3)
- added C169: 0.1uF, Capacitor_SMD:C_0402_1005Metric, F.Cu at (25.9, 14.3)
- added C17: 0.22uF, Capacitor_SMD:C_0402_1005Metric, F.Cu at (-8.93, 25.8)
- added C170: 0.1uF, Capacitor_SMD:C_0402_1005Metric, F.Cu at (25.9, 16.2)
- added C171: 10uF, Capacitor_SMD:C_0402_1005Metric, F.Cu at (28.8, 0.48)
- added C172: 22uF, Capacitor_SMD:C_0402_1005Metric, F.Cu at (28.8, 2.46)
- added C173: 0.1uF, Capacitor_SMD:C_0402_1005Metric, F.Cu at (28.8, 4.42)
- added C174: 0.1uF, Capacitor_SMD:C_0402_1005Metric, F.Cu at (28.8, 6.39)
- added C175: 10uF, Capacitor_SMD:C_0402_1005Metric, F.Cu at (28.8, 8.37)
- added C176: 22uF, Capacitor_SMD:C_0402_1005Metric, F.Cu at (28.8, 10.3)
- added C177: 0.1uF, Capacitor_SMD:C_0402_1005Metric, F.Cu at (28.8, 12.3)
- added C178: 0.1uF, Capacitor_SMD:C_0402_1005Metric, F.Cu at (28.8, 14.3)
- added C179: 10uF, Capacitor_SMD:C_0402_1005Metric, F.Cu at (28.8, 16.2)
- added C18: 0.22uF, Capacitor_SMD:C_0402_1005Metric, F.Cu at (-8.93, 27.8)
- added C180: 22uF, Capacitor_SMD:C_0402_1005Metric, F.Cu at (31.6, 0.48)
- added C181: 0.1uF, Capacitor_SMD:C_0402_1005Metric, F.Cu at (31.6, 2.46)
- added C182: 10uF, Capacitor_SMD:C_0402_1005Metric, F.Cu at (31.6, 4.42)
- added C183: 22uF, Capacitor_SMD:C_0402_1005Metric, F.Cu at (31.6, 6.39)
- added C184: 0.1uF, Capacitor_SMD:C_0402_1005Metric, F.Cu at (31.6, 8.37)
- added C185: 22uF, Capacitor_SMD:C_0402_1005Metric, F.Cu at (31.6, 10.3)
- added C186: 0.1uF, Capacitor_SMD:C_0402_1005Metric, F.Cu at (31.6, 12.3)
- added C187: 4.7uF, Capacitor_SMD:C_0402_1005Metric, F.Cu at (31.6, 14.3)
- added C188: 22uF, Capacitor_SMD:C_0402_1005Metric, F.Cu at (31.6, 16.2)
- added C189: 0.1uF, Capacitor_SMD:C_0402_1005Metric, F.Cu at (34.5, 0.48)
- added C19: 0.22uF, Capacitor_SMD:C_0402_1005Metric, F.Cu at (-8.93, 29.8)
- added C190: 4.7uF, Capacitor_SMD:C_0402_1005Metric, F.Cu at (34.5, 2.46)
- added C191: 22uF, Capacitor_SMD:C_0402_1005Metric, F.Cu at (34.5, 4.42)
- added C192: 0.1uF, Capacitor_SMD:C_0402_1005Metric, F.Cu at (34.5, 6.39)
- added C193: 22uF, Capacitor_SMD:C_0402_1005Metric, F.Cu at (34.5, 8.37)
- added C194: 0.1uF, Capacitor_SMD:C_0402_1005Metric, F.Cu at (34.5, 10.3)
- added C20: 0.22uF, Capacitor_SMD:C_0402_1005Metric, F.Cu at (-8.93, 31.7)
- added C21: 0.22uF, Capacitor_SMD:C_0402_1005Metric, F.Cu at (-8.93, 33.7)
- added C22: 0.22uF, Capacitor_SMD:C_0402_1005Metric, F.Cu at (-8.93, 35.7)
- added C23: 0.22uF, Capacitor_SMD:C_0402_1005Metric, F.Cu at (-8.93, 37.6)
- added C24: 0.22uF, Capacitor_SMD:C_0402_1005Metric, F.Cu at (-8.93, 39.6)
- added C25: 0.22uF, Capacitor_SMD:C_0402_1005Metric, F.Cu at (-8.93, 41.6)
- added C26: 0.22uF, Capacitor_SMD:C_0402_1005Metric, F.Cu at (-6.05, 21.9)
- added C27: 0.22uF, Capacitor_SMD:C_0402_1005Metric, F.Cu at (-6.05, 23.8)
- added C28: 0.22uF, Capacitor_SMD:C_0402_1005Metric, F.Cu at (-6.05, 25.8)
- added C29: 0.22uF, Capacitor_SMD:C_0402_1005Metric, F.Cu at (-6.05, 27.8)
- added C30: 0.22uF, Capacitor_SMD:C_0402_1005Metric, F.Cu at (-6.05, 29.8)
- added C31: 0.22uF, Capacitor_SMD:C_0402_1005Metric, F.Cu at (-6.05, 31.7)
- added C32: 0.22uF, Capacitor_SMD:C_0402_1005Metric, F.Cu at (-6.05, 33.7)
- added C33: 0.22uF, Capacitor_SMD:C_0402_1005Metric, F.Cu at (-6.05, 35.7)
- added C34: 0.22uF, Capacitor_SMD:C_0402_1005Metric, F.Cu at (-6.05, 37.6)
- added C35: 0.22uF, Capacitor_SMD:C_0402_1005Metric, F.Cu at (-6.05, 39.6)
- added C36: 0.22uF, Capacitor_SMD:C_0402_1005Metric, F.Cu at (-6.05, 41.6)
- added C37: 0.22uF, Capacitor_SMD:C_0402_1005Metric, F.Cu at (-3.19, 21.9)
- added C38: 0.22uF, Capacitor_SMD:C_0402_1005Metric, F.Cu at (-3.19, 23.8)
- added C39: 0.22uF, Capacitor_SMD:C_0402_1005Metric, F.Cu at (-3.19, 25.8)
- added C40: 0.22uF, Capacitor_SMD:C_0402_1005Metric, F.Cu at (-3.19, 27.8)
- added C41: 0.22uF, Capacitor_SMD:C_0402_1005Metric, F.Cu at (-3.19, 29.8)
- added C42: 0.22uF, Capacitor_SMD:C_0402_1005Metric, F.Cu at (-3.19, 31.7)
- added C43: 0.22uF, Capacitor_SMD:C_0402_1005Metric, F.Cu at (-3.19, 33.7)
- added C44: 0.22uF, Capacitor_SMD:C_0402_1005Metric, F.Cu at (-3.19, 35.7)
- added C45: 0.22uF, Capacitor_SMD:C_0402_1005Metric, F.Cu at (-3.19, 37.6)
- added C46: 0.22uF, Capacitor_SMD:C_0402_1005Metric, F.Cu at (-3.19, 39.6)
- added C47: 0.22uF, Capacitor_SMD:C_0402_1005Metric, F.Cu at (-3.19, 41.6)
- added C48: 0.22uF, Capacitor_SMD:C_0402_1005Metric, F.Cu at (-0.32, 21.9)
- added C49: 0.22uF, Capacitor_SMD:C_0402_1005Metric, F.Cu at (-0.32, 23.8)
- added C50: 0.22uF, Capacitor_SMD:C_0402_1005Metric, F.Cu at (-0.32, 25.8)
- added C51: 0.22uF, Capacitor_SMD:C_0402_1005Metric, F.Cu at (-0.32, 27.8)
- added C52: 0.22uF, Capacitor_SMD:C_0402_1005Metric, F.Cu at (-0.32, 29.8)
- added C53: 0.22uF, Capacitor_SMD:C_0402_1005Metric, F.Cu at (-0.32, 31.7)
- added C54: 0.22uF, Capacitor_SMD:C_0402_1005Metric, F.Cu at (-0.32, 33.7)
- added C55: 0.22uF, Capacitor_SMD:C_0402_1005Metric, F.Cu at (-0.32, 35.7)
- added C56: 0.22uF, Capacitor_SMD:C_0402_1005Metric, F.Cu at (-0.32, 37.6)
- added C57: 0.22uF, Capacitor_SMD:C_0402_1005Metric, F.Cu at (-0.32, 39.6)
- added C58: 0.22uF, Capacitor_SMD:C_0402_1005Metric, F.Cu at (-0.32, 41.6)
- added C59: 0.22uF, Capacitor_SMD:C_0402_1005Metric, F.Cu at (2.56, 21.9)
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Connections:
- net VL805_0_PE_RX_C_N renamed FT_PEU0_X1_C_RXN0
- net VL805_0_PE_RX_C_P renamed FT_PEU0_X1_C_RXP0
- C1 pad 1: VL805_0_PE_RX_P -> FT_PEU0_X1_RXP0
- C2 pad 1: VL805_0_PE_RX_N -> FT_PEU0_X1_RXN0
- C7 pad 1: VL805_1_PE_RX_P -> unconnected-(C7-Pad1)
- C7 pad 2: VL805_1_PE_RX_C_P -> unconnected-(C7-Pad2)
- U3 pad A10: unconnected-(U3F-LMU0_DQ48-PadA10) -> FT_MEM0_DQ48
- U3 pad A11: unconnected-(U3F-LMU0_DQS_C15-PadA11) -> FT_MEM0_DQS_C_15
- U3 pad A12: unconnected-(U3F-LMU0_DQ55-PadA12) -> FT_MEM0_DQ55
- U3 pad A13: unconnected-(U3F-LMU0_DQ51-PadA13) -> FT_MEM0_DQ51
- U3 pad A14: unconnected-(U3F-LMU0_DQ32-PadA14) -> FT_MEM0_DQ32
- U3 pad A15: unconnected-(U3F-LMU0_DQS_C13-PadA15) -> FT_MEM0_DQS_C_13
- U3 pad A16: unconnected-(U3F-LMU0_DQ38-PadA16) -> FT_MEM0_DQ38
- U3 pad A17: unconnected-(U3F-LMU0_DQ34-PadA17) -> FT_MEM0_DQ34
- U3 pad A18: unconnected-(U3F-LMU0_CB0-PadA18) -> FT_MEM0_DQ64
- U3 pad A19: unconnected-(U3F-LMU0_DQS_C17-PadA19) -> FT_MEM0_DQS_C_17
- U3 pad A20: unconnected-(U3F-LMU0_CB7-PadA20) -> FT_MEM0_DQ71
- U3 pad A21: unconnected-(U3F-LMU0_CB1-PadA21) -> FT_MEM0_DQ65
- U3 pad A23: unconnected-(U3F-LMU0_A9-PadA23) -> FT_MEM0_A9
- U3 pad A25: unconnected-(U3F-LMU0_A3-PadA25) -> FT_MEM0_A3
- U3 pad A28: unconnected-(U3F-LMU0_PAR-PadA28) -> FT_MEM0_PAR
- U3 pad A3: unconnected-(U3E-PEU1_X16_TXP0-PadA3) -> (no net)
- U3 pad A31: unconnected-(U3F-LMU0_A17-PadA31) -> FT_MEM0_A17
- U3 pad A4: unconnected-(U3E-PEU1_X16_TXN0-PadA4) -> (no net)
- U3 pad A7: unconnected-(U3E-PEU1_X16_RXP0-PadA7) -> (no net)
- U3 pad A8: unconnected-(U3E-PEU1_X16_RXN0-PadA8) -> (no net)
- U3 pad AA10: unconnected-(U3B-VDD-PadAA10) -> (no net)
- U3 pad AA12: unconnected-(U3B-PEU0_AVDDCLK-PadAA12) -> (no net)
- U3 pad AA13: unconnected-(U3E-PEU0_X1_REXT-PadAA13) -> (no net)
- U3 pad AA14: unconnected-(U3B-VDD-PadAA14) -> (no net)
- U3 pad AA16: +1V2 -> (no net)
- U3 pad AA17: unconnected-(U3F-LMU1_BP_ZN-PadAA17) -> Net-(U3F-LMU1_BP_ZN)
- U3 pad AA18: +1V2 -> (no net)
- U3 pad AA21: unconnected-(U3B-RSVD30_FLOAT-PadAA21) -> (no net)
- U3 pad AA23: +1V8 -> (no net)
- U3 pad AA24: +1V2 -> GND
- U3 pad AA26: unconnected-(U3E-PEU1_REFCLKP-PadAA26) -> (no net)
- U3 pad AA27: +1V2 -> (no net)
- U3 pad AA28: unconnected-(U3C-RSVD31_FLOAT-PadAA28) -> (no net)
- U3 pad AA29: unconnected-(U3C-CAN_TX0/PEU1_LINKUP1-PadAA29) -> (no net)
- U3 pad AA3: unconnected-(U3E-PEU0_X16_TXN12-PadAA3) -> (no net)
- U3 pad AA31: unconnected-(U3F-LMU1_DQ2-PadAA31) -> FT_MEM1_DQ2
- U3 pad AA32: unconnected-(U3F-LMU1_DQ15-PadAA32) -> FT_MEM1_DQ15
- U3 pad AA34: unconnected-(U3F-LMU1_DQ12-PadAA34) -> FT_MEM1_DQ12
- U3 pad AA4: unconnected-(U3E-PEU0_X16_TXP12-PadAA4) -> (no net)
- U3 pad AA7: NVME_PE_RX3_P -> (no net)
- U3 pad AA8: NVME_PE_RX3_N -> (no net)
- U3 pad AB1: NVME_PE_TX3_P -> (no net)
- U3 pad AB10: unconnected-(U3E-PEU0_X1_ATB1-PadAB10) -> (no net)
- U3 pad AB11: unconnected-(U3B-PEU0_AVDD-PadAB11) -> (no net)
- U3 pad AB13: +1V8 -> (no net)
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Routing:
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Other:
- outline, holes or cut-outs redrawn

Commit message: update schem + pcb layout
Parts:
- removed the J3 at (288.5, 16.1)
- removed the J3 at (268.0, 16.1)
- removed J8: RJ45_RB1-125B8G1A, Connector_RJ:RJ45_UDE_RB1-125B8G1A
- removed the REF** at (168.5, 77.9)
- removed the REF** at (196.5, 77.9)
- added C195: 0.1uF, Capacitor_SMD:C_0402_1005Metric, F.Cu at (16.4, 67.1)
- added C196: 0.1uF, Capacitor_SMD:C_0402_1005Metric, F.Cu at (19.3, 63.1)
- added C197: 4.7uF, Capacitor_SMD:C_0603_1608Metric, F.Cu at (26.8, 51.5)
- added C198: 270uF, Capacitor_Tantalum_SMD:CP_EIA-7361-38_AVX-V, F.Cu at (93.5, 65.0)
- added C199: 270uF, Capacitor_Tantalum_SMD:CP_EIA-7361-38_AVX-V, F.Cu at (19.9, 58.3)
- added C200: 4.7uF, Capacitor_SMD:C_0603_1608Metric, F.Cu at (26.8, 54.0)
- added C201: 0.1uF, Capacitor_SMD:C_0603_1608Metric, F.Cu at (26.8, 56.5)
- added C202: 0.1uF, Capacitor_SMD:C_0603_1608Metric, F.Cu at (26.8, 59.0)
- added C203: 0.1uF, Capacitor_SMD:C_0603_1608Metric, F.Cu at (26.8, 61.5)
- added C204: 0.1uF, Capacitor_SMD:C_0603_1608Metric, F.Cu at (26.8, 64.0)
- added C205: 4.7uF, Capacitor_SMD:C_1206_3216Metric, F.Cu at (27.6, 48.5)
- added C206: 0.1uF, Capacitor_SMD:C_0402_1005Metric, F.Cu at (19.3, 65.1)
- added C207: 0.1uF, Capacitor_SMD:C_0402_1005Metric, F.Cu at (19.3, 67.1)
- added C208: 0.1uF, Capacitor_SMD:C_0402_1005Metric, F.Cu at (22.1, 63.1)
- added C209: 0.1uF, Capacitor_SMD:C_0402_1005Metric, F.Cu at (22.1, 65.1)
- added C210: 0.1uF, Capacitor_SMD:C_0402_1005Metric, F.Cu at (22.1, 67.1)
- added C211: 270uF, Capacitor_SMD:C_1206_3216Metric, F.Cu at (17.8, 71.7)
- added C212: 270uF, Capacitor_SMD:C_1206_3216Metric, F.Cu at (17.8, 75.1)
- added C213: 270uF, Capacitor_SMD:C_1206_3216Metric, F.Cu at (17.8, 78.4)
- added C214: 270uF, Capacitor_SMD:C_1206_3216Metric, F.Cu at (17.8, 81.8)
- added C215: 1uF, Capacitor_SMD:C_0402_1005Metric, F.Cu at (28.0, 31.9)
- added C216: 100pF, Capacitor_SMD:C_0402_1005Metric, F.Cu at (28.0, 33.9)
- added C217: 22uF, Capacitor_SMD:C_0603_1608Metric, F.Cu at (17.0, 17.1)
- added C218: 22uF, Capacitor_SMD:C_0603_1608Metric, F.Cu at (17.0, 19.6)
- added C219: 22uF, Capacitor_SMD:C_0603_1608Metric, F.Cu at (17.0, 22.1)
- added C220: 4.7uF, Capacitor_SMD:C_0603_1608Metric, F.Cu at (17.0, 24.6)
- added C221: 4.7uF, Capacitor_SMD:C_0603_1608Metric, F.Cu at (17.0, 27.1)
- added C222: 0.1uF, Capacitor_SMD:C_0603_1608Metric, F.Cu at (17.0, 29.7)
- added C223: 0.22uF, Capacitor_SMD:C_0603_1608Metric, F.Cu at (21.0, 17.1)
- added C224: 47uF, Capacitor_SMD:C_1206_3216Metric, B.Cu at (299.5, 168.0)
- added C225: 47uF, Capacitor_SMD:C_1206_3216Metric, B.Cu at (299.5, 165.5)
- added C226: 47uF, Capacitor_SMD:C_1206_3216Metric, B.Cu at (299.5, 163.0)
- added C227: 47uF, Capacitor_SMD:C_1206_3216Metric, F.Cu at (299.5, 163.0)
- added C228: 10uF, Capacitor_SMD:C_0603_1608Metric, F.Cu at (21.0, 19.6)
- added C229: 10uF, Capacitor_SMD:C_0603_1608Metric, F.Cu at (21.0, 22.1)
- added C230: 0.1uF, Capacitor_SMD:C_0603_1608Metric, F.Cu at (21.0, 24.6)
- added C231: 0.1uF, Capacitor_SMD:C_0603_1608Metric, F.Cu at (21.0, 27.1)
- added C232: 560uF, Capacitor_SMD:CP_Elec_6.3x5.9, F.Cu at (309.5, 158.0)
- added C233: 560uF, Capacitor_SMD:CP_Elec_6.3x5.9, F.Cu at (309.0, 168.0)
- added C234: 560uF, Capacitor_SMD:CP_Elec_6.3x5.9, F.Cu at (317.5, 158.0)
- added C235: 2.2nF, Capacitor_SMD:C_0603_1608Metric, F.Cu at (21.0, 29.7)
- added C236: 10nF (NC), Capacitor_SMD:C_0603_1608Metric, F.Cu at (25.0, 17.1)
- added C237: 22uF, Capacitor_SMD:C_0603_1608Metric, F.Cu at (25.0, 19.6)
- added C238: 22uF, Capacitor_SMD:C_0603_1608Metric, F.Cu at (25.0, 22.1)
- added C239: 4.7uF, Capacitor_SMD:C_0603_1608Metric, F.Cu at (25.0, 24.6)
- added C240: 4.7uF, Capacitor_SMD:C_0603_1608Metric, F.Cu at (25.0, 27.1)
- added C241: 22uF, Capacitor_SMD:C_0603_1608Metric, F.Cu at (25.0, 29.7)
- added C242: 0.1uF, Capacitor_SMD:C_0603_1608Metric, F.Cu at (29.0, 17.1)
- added C243: 100pF, Capacitor_SMD:C_0402_1005Metric, F.Cu at (28.0, 35.8)
- added C244: 1uF, Capacitor_SMD:C_0402_1005Metric, F.Cu at (28.0, 37.8)
- added C245: 0.22uF, Capacitor_SMD:C_0603_1608Metric, F.Cu at (29.0, 19.6)
- added C246: 47uF, Capacitor_SMD:C_1206_3216Metric, F.Cu at (299.5, 160.5)
- added C247: 47uF, Capacitor_SMD:C_1206_3216Metric, F.Cu at (299.5, 165.5)
- added C248: 47uF, Capacitor_SMD:C_1206_3216Metric, B.Cu at (299.5, 160.5)
- added C249: 47uF, Capacitor_SMD:C_1206_3216Metric, F.Cu at (299.5, 168.0)
- added C250: 10uF, Capacitor_SMD:C_0603_1608Metric, F.Cu at (29.0, 22.1)
- added C251: 22uF, Capacitor_SMD:C_0402_1005Metric, F.Cu at (24.9, 71.0)
- added C252: 10uF, Capacitor_SMD:C_0603_1608Metric, F.Cu at (29.0, 24.6)
- added C253: 0.1uF, Capacitor_SMD:C_0603_1608Metric, F.Cu at (29.0, 27.1)
- added C254: 22uF, Capacitor_SMD:C_0402_1005Metric, F.Cu at (24.9, 73.0)
- added C255: 0.1uF, Capacitor_SMD:C_0603_1608Metric, F.Cu at (29.0, 29.7)
- added C256: 22uF, Capacitor_SMD:C_0402_1005Metric, F.Cu at (24.9, 75.0)
- added C257: 22uF, Capacitor_SMD:C_0402_1005Metric, F.Cu at (24.9, 77.0)
- added C258: 1uF, Capacitor_SMD:C_0402_1005Metric, F.Cu at (24.9, 78.9)
- added C259: 1uF, Capacitor_SMD:C_0402_1005Metric, F.Cu at (24.9, 80.9)
- added C261: 1uF, Capacitor_SMD:C_0402_1005Metric, F.Cu at (74.9, 29.4)
- added C262: 22uF, Capacitor_SMD:C_0603_1608Metric, F.Cu at (75.5, 17.1)
- added C263: 22uF, Capacitor_SMD:C_0603_1608Metric, F.Cu at (75.5, 19.6)
- added C264: 22uF, Capacitor_SMD:C_0603_1608Metric, F.Cu at (75.5, 22.1)
- added C265: 0.22uF, Capacitor_SMD:C_0402_1005Metric, F.Cu at (74.9, 31.4)
- added C266: 560uF, Capacitor_SMD:C_1206_3216Metric, F.Cu at (67.7, 17.5)
- added C267: 22uF, Capacitor_SMD:C_0603_1608Metric, F.Cu at (75.5, 24.6)
- added C268: 22uF, Capacitor_SMD:C_0603_1608Metric, F.Cu at (75.5, 27.1)
- added C269: 22uF, Capacitor_SMD:C_0603_1608Metric, F.Cu at (79.5, 17.1)
- added C270: 22uF, Capacitor_SMD:C_0603_1608Metric, F.Cu at (79.5, 19.6)
- added C271: 22uF, Capacitor_SMD:C_0603_1608Metric, F.Cu at (79.5, 22.1)
- added C272: 22uF, Capacitor_SMD:C_0603_1608Metric, F.Cu at (79.5, 24.6)
- added C273: 0.22uF, Capacitor_SMD:C_0402_1005Metric, F.Cu at (74.9, 33.3)
- added C274: 47uF, Capacitor_SMD:C_1206_3216Metric, F.Cu at (67.7, 20.9)
- added C275: 47uF, Capacitor_SMD:C_1206_3216Metric, F.Cu at (67.7, 24.2)
- added C276: 47uF, Capacitor_SMD:C_1206_3216Metric, F.Cu at (67.7, 27.6)
- added C277: 47uF, Capacitor_SMD:C_1206_3216Metric, F.Cu at (67.7, 30.9)
- added C278: 10uF, Capacitor_SMD:C_0603_1608Metric, F.Cu at (79.5, 27.1)
- added C279: 10uF, Capacitor_SMD:C_0603_1608Metric, F.Cu at (83.5, 17.1)
- added C280: 10uF, Capacitor_SMD:C_0603_1608Metric, F.Cu at (83.5, 19.6)
- added C281: 10uF, Capacitor_SMD:C_0603_1608Metric, F.Cu at (83.5, 22.1)
- added C93: 0.1uF, Capacitor_SMD:C_0402_1005Metric, F.Cu at (16.4, 63.1)
- added C94: 0.1uF, Capacitor_SMD:C_0402_1005Metric, F.Cu at (16.4, 65.1)
- added D1: LIFE_LED, LED_SMD:LED_0603_1608Metric, F.Cu at (31.5, 36.8)
- added D2: LED, LED_SMD:LED_0603_1608Metric, F.Cu at (28.4, 74.8)
- added D3: LED, LED_SMD:LED_0603_1608Metric, F.Cu at (28.4, 77.4)
- added H1: MountingHole, MountingHole:MountingHole_3.2mm_M3_Pad, F.Cu at (65.4, 43.5)
- added H2: MountingHole, MountingHole:MountingHole_3.2mm_M3_Pad, F.Cu at (65.4, 51.5)
- added H3: MountingHole, MountingHole:MountingHole_3.2mm_M3_Pad, F.Cu at (73.3, 43.5)
- added H4: MountingHole, MountingHole:MountingHole_3.2mm_M3_Pad, F.Cu at (73.3, 51.5)
- added IC1: USB7016_KDX, USB7016_KDX:QFN40P1200X1200X90-101N-D, F.Cu at (307.2, 97.3)
- added IC1: AP61300Z6-7, AP61300Z6-7:SOTFL50P162X60-6N, F.Cu at (16.7, 85.0)
- added J10: 39-29-9042, 39-29-9042:39-29-904Y, F.Cu at (324.5, 112.9)
- added J11: M.2_NVME1, m.2-m1_2199119_5:TE_1-2199119-5, F.Cu at (205.0, 144.6)
- added J12: USB3_A0, Connector_USB:USB_A_Receptacle_XKB_U231-091N-4BLRA00-S, F.Cu at (304.4, 74.1)
- added J13: USB3_A1, Connector_USB:USB_A_Receptacle_XKB_U231-091N-4BLRA00-S, F.Cu at (286.9, 74.2)
- added J3: Micro_SD_Card, Connector_Card:microSD_HC_Wuerth_693072010801, F.Cu at (206.4, 72.8)
- added L1: 0.22uH, Inductor_SMD:L_APV_APH1050, F.Cu at (311.0, 145.5)
- added L2: 0.22uH, Inductor_SMD:L_APV_APH1050, F.Cu at (322.5, 145.5)
- added L3: 1uH, Inductor_SMD:L_1206_3216Metric, F.Cu at (29.3, 71.8)
- added MH8: TEST_POINT_TH_200_112_NN, TH_200_112, F.Cu at (192.0, 153.5)
- added MH8: TEST_POINT_TH_200_112_NN, TH_200_112, F.Cu at (192.0, 143.5)
- added MH8: TEST_POINT_TH_200_112_NN, TH_200_112, F.Cu at (192.0, 105.5)
- added MH8: TEST_POINT_TH_200_112_NN, TH_200_112, F.Cu at (192.0, 115.5)
- added Q1: 2N7002, Package_TO_SOT_SMD:SOT-23, F.Cu at (28.8, 85.7)
- added Q2: 2N7002, Package_TO_SOT_SMD:SOT-23, F.Cu at (31.9, 33.3)
- added R100: 10k, Resistor_SMD:R_0402_1005Metric, F.Cu at (72.0, 26.8)
- added R101: 10k, Resistor_SMD:R_0402_1005Metric, F.Cu at (72.0, 28.8)
- added R48: 4.7k, Resistor_SMD:R_0402_1005Metric, F.Cu at (22.1, 71.0)
- added R49: 4.7k, Resistor_SMD:R_0402_1005Metric, F.Cu at (22.1, 73.0)
- added R50: 0r (NC), Resistor_SMD:R_0402_1005Metric, F.Cu at (85.0, 87.0)
- added R51: 0.01r, Resistor_SMD:R_0402_1005Metric, F.Cu at (16.4, 31.9)
- added R52: 4.7k, Resistor_SMD:R_0402_1005Metric, F.Cu at (30.2, 51.2)
- added R53: 4.7k, Resistor_SMD:R_0402_1005Metric, F.Cu at (30.2, 53.2)
- added R54: 4.7k, Resistor_SMD:R_0402_1005Metric, F.Cu at (30.2, 55.2)
- added R55: 0r, Resistor_SMD:R_0402_1005Metric, F.Cu at (30.2, 57.2)
- added R56: 0r, Resistor_SMD:R_0402_1005Metric, F.Cu at (30.2, 59.1)
- added R57: 0r, Resistor_SMD:R_0402_1005Metric, F.Cu at (30.2, 61.1)
- added R58: 0r, Resistor_SMD:R_0402_1005Metric, F.Cu at (30.2, 63.1)
- added R59: 4.7k, Resistor_SMD:R_0402_1005Metric, F.Cu at (30.2, 65.1)
- added R60: 0r, Resistor_SMD:R_0402_1005Metric, F.Cu at (16.4, 33.9)
- added R61: 0r, Resistor_SMD:R_0402_1005Metric, F.Cu at (16.4, 35.9)
- added R62: 0r (NC), Resistor_SMD:R_0402_1005Metric, F.Cu at (16.4, 37.9)
- added R63: 2.2r, Resistor_SMD:R_0603_1608Metric, F.Cu at (33.0, 17.1)
- added R64: 60.4k, Resistor_SMD:R_0603_1608Metric, F.Cu at (33.0, 19.6)
- added R65: 0r, Resistor_SMD:R_0402_1005Metric, F.Cu at (16.4, 39.9)
- added R66: 100k, Resistor_SMD:R_0402_1005Metric, F.Cu at (16.4, 41.9)
- added R67: 10k, Resistor_SMD:R_0402_1005Metric, F.Cu at (16.4, 43.9)
- added R68: 10k, Resistor_SMD:R_0402_1005Metric, F.Cu at (19.3, 31.9)
- added R69: 10k, Resistor_SMD:R_0402_1005Metric, F.Cu at (19.3, 33.9)
- added R70: 0r, Resistor_SMD:R_0402_1005Metric, F.Cu at (19.3, 35.9)
- added R71: 30.1k, Resistor_SMD:R_0402_1005Metric, F.Cu at (19.3, 37.9)
- added R72: 0r, Resistor_SMD:R_0402_1005Metric, F.Cu at (19.3, 39.9)
- added R73: 0r, Resistor_SMD:R_0402_1005Metric, F.Cu at (19.3, 41.9)
- added R74: 10k, Resistor_SMD:R_0402_1005Metric, F.Cu at (19.3, 43.9)
- added R75: 4.7k, Resistor_SMD:R_0402_1005Metric, F.Cu at (22.2, 31.9)
- added R76: 0r, Resistor_SMD:R_0402_1005Metric, F.Cu at (22.2, 33.9)
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Connections:
- net /BOOT renamed /CPLD/BOOT
- net /R_D+ renamed /CPLD/R_D+
- net /R_D- renamed /CPLD/R_D-
- net VL805_0_PE_CLK_N renamed FT_PEU0_VL805_CLK_N
- net VL805_0_PE_CLK_P renamed FT_PEU0_VL805_CLK_P
- net VL805_1_PE_RX_C_N renamed FT_PEU1_X1_C_RXN0
- C7 pad 1: unconnected-(C7-Pad1) -> FT_PEU1_X1_RXP0
- C7 pad 2: unconnected-(C7-Pad2) -> FT_PEU1_X1_C_RXP0
- C8 pad 1: VL805_1_PE_RX_N -> FT_PEU1_X1_RXN0
- C90 pad 2: VREF_CA1 -> VREF_CA0
- CN2 pad 1: unconnected-(CN2-Pad1) -> 3V3_ATX
- CN2 pad 10: unconnected-(CN2-Pad10) -> 12V_ATX
- CN2 pad 11: unconnected-(CN2-Pad11) -> 12V_ATX
- CN2 pad 12: unconnected-(CN2-Pad12) -> 3V3_ATX
- CN2 pad 13: unconnected-(CN2-Pad13) -> 3V3_ATX
- CN2 pad 14: unconnected-(CN2-Pad14) -> -12V_ATX
- CN2 pad 15: unconnected-(CN2-Pad15) -> GND
- CN2 pad 16: unconnected-(CN2-Pad16) -> PS_ON_ATX
- CN2 pad 17: unconnected-(CN2-Pad17) -> GND
- CN2 pad 18: unconnected-(CN2-Pad18) -> GND
- CN2 pad 19: unconnected-(CN2-Pad19) -> GND
- CN2 pad 2: unconnected-(CN2-Pad2) -> 3V3_ATX
- CN2 pad 21: unconnected-(CN2-Pad21) -> 5V_ATX
- CN2 pad 22: unconnected-(CN2-Pad22) -> 5V_ATX
- CN2 pad 23: unconnected-(CN2-Pad23) -> 5V_ATX
- CN2 pad 24: unconnected-(CN2-Pad24) -> GND
- CN2 pad 3: unconnected-(CN2-Pad3) -> Net-(CN2-Pad3)
- CN2 pad 4: unconnected-(CN2-Pad4) -> 5V_ATX
- CN2 pad 5: unconnected-(CN2-Pad5) -> Net-(CN2-Pad3)
- CN2 pad 6: unconnected-(CN2-Pad6) -> 5V_ATX
- CN2 pad 7: unconnected-(CN2-Pad7) -> Net-(CN2-Pad3)
- CN2 pad 8: unconnected-(CN2-Pad8) -> PWRGD_ATX
- CN2 pad 9: unconnected-(CN2-Pad9) -> 5V_STBY_ATX
- J4 pad 1: Net-(J4-GND-Pad1) -> GND
- J4 pad 10: unconnected-(J4-DAS/~{DSS}/~{LED1}-Pad10) -> M2_LED0
- J4 pad 11: NVME_PE_TX3_P -> FT_PEU0_TXN11
- J4 pad 2: Net-(J4-3.3V-Pad12) -> 3V3
- J4 pad 21: Net-(J4-GND-Pad1) -> GND
- J4 pad 23: NVME_PE_TX2_P -> FT_PEU0_TXN10
- J4 pad 25: NVME_PE_TX2_N -> FT_PEU0_TXP10
- J4 pad 27: Net-(J4-GND-Pad1) -> GND
- J4 pad 29: NVME_PE_RX1_P -> FT_PEU0_RXN9
- J4 pad 3: Net-(J4-GND-Pad1) -> GND
- J4 pad 31: NVME_PE_RX1_N -> FT_PEU0_RXP9
- J4 pad 33: Net-(J4-GND-Pad1) -> GND
- J4 pad 35: NVME_PE_TX1_P -> FT_PEU0_TXN9
- J4 pad 37: NVME_PE_TX1_N -> FT_PEU0_TXP9
- J4 pad 39: Net-(J4-GND-Pad1) -> GND
- J4 pad 4: Net-(J4-3.3V-Pad12) -> 3V3
- J4 pad 41: NVME_PE_RX0_P -> FT_PEU0_RXN8
- J4 pad 43: NVME_PE_RX0_N -> FT_PEU0_RXP8
- J4 pad 45: Net-(J4-GND-Pad1) -> GND
- J4 pad 47: NVME_PE_TX0_P -> FT_PEU0_TXN8
- J4 pad 49: NVME_PE_TX0_N -> FT_PEU0_TXP8
- J4 pad 5: NVME_PE_RX3_P -> FT_PEU0_RXN11
- J4 pad 50: unconnected-(J4-~{PERST}-Pad50) -> FT_PCIE_NVME_RST
- J4 pad 51: Net-(J4-GND-Pad1) -> GND
- J4 pad 53: unconnected-(J4-REFCLKn-Pad53) -> Net-(J4-REFCLKn)
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Routing:
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
Commit message: update schem + pcb layout
Parts:
- removed the H1 at (163.0, 232.5)
- removed the H2 at (321.0, 232.5)
- removed the H3 at (163.2, 77.1)
- removed the H4 at (321.0, 100.0)
- removed MH8 (x4): TEST_POINT_TH_200_112_NN, TH_200_112
- added C260: 18pF, Capacitor_SMD:C_0402_1005Metric, F.Cu at (20.6, 45.3)
- added C282: 18pF, Capacitor_SMD:C_0402_1005Metric, F.Cu at (20.6, 47.2)
- added C283: 0.1uF, Capacitor_SMD:C_0402_1005Metric, F.Cu at (20.6, 49.2)
- added C284: 0.1uF, Capacitor_SMD:C_0402_1005Metric, F.Cu at (20.6, 51.2)
- added C285: 0.1uF, Capacitor_SMD:C_0402_1005Metric, F.Cu at (20.6, 53.1)
- added C286: 0.1uF, Capacitor_SMD:C_0402_1005Metric, F.Cu at (23.4, 41.3)
- added C287: 0.1uF, Capacitor_SMD:C_0402_1005Metric, F.Cu at (23.4, 43.3)
- added C288: 0.1uF, Capacitor_SMD:C_0402_1005Metric, F.Cu at (23.4, 45.3)
- added C289: 0.1uF, Capacitor_SMD:C_0402_1005Metric, F.Cu at (23.4, 47.2)
- added C290: 0.1uF, Capacitor_SMD:C_0402_1005Metric, F.Cu at (23.4, 49.2)
- added C291: 0.1uF, Capacitor_SMD:C_0402_1005Metric, F.Cu at (23.4, 51.2)
- added C292: 0.1uF, Capacitor_SMD:C_0402_1005Metric, F.Cu at (23.4, 53.1)
- added C293: 0.1uF, Capacitor_SMD:C_0402_1005Metric, F.Cu at (26.3, 41.3)
- added C294: 0.1uF, Capacitor_SMD:C_0402_1005Metric, F.Cu at (26.3, 43.3)
- added C295: 0.1uF, Capacitor_SMD:C_0402_1005Metric, F.Cu at (26.3, 45.3)
- added C296: 0.1uF, Capacitor_SMD:C_0402_1005Metric, F.Cu at (26.3, 47.2)
- added C297: 0.1uF, Capacitor_SMD:C_0402_1005Metric, F.Cu at (26.3, 49.2)
- added CN3: APCI0079-P002A, LOTES-APCI0079-P002A-M.2:PCI-SMD_APCI0079-P002A, F.Cu at (208.1, 219.3)
- added Q3: 2N7002, Package_TO_SOT_SMD:SOT-23, F.Cu at (46.0, 90.5)
- added R102: 560r, Resistor_SMD:R_0402_1005Metric, F.Cu at (56.5, 86.9)
- added R103: 560r, Resistor_SMD:R_0402_1005Metric, F.Cu at (56.5, 88.9)
- added R104: 10k, Resistor_SMD:R_0402_1005Metric, F.Cu at (80.1, 19.7)
- added R105: 10k, Resistor_SMD:R_0402_1005Metric, F.Cu at (80.1, 21.6)
- added R106: 10k, Resistor_SMD:R_0402_1005Metric, F.Cu at (80.1, 23.6)
- added R107: 0r, Resistor_SMD:R_0402_1005Metric, F.Cu at (80.1, 25.6)
- added R108: 10k, Resistor_SMD:R_0402_1005Metric, F.Cu at (80.1, 27.6)
- added R109: 4.7k, Resistor_SMD:R_0402_1005Metric, F.Cu at (20.6, 57.1)
- added R110: 4.7k, Resistor_SMD:R_0402_1005Metric, F.Cu at (20.6, 59.1)
- added R111: 4.7k, Resistor_SMD:R_0402_1005Metric, F.Cu at (20.6, 61.1)
- added R112: 4.7k, Resistor_SMD:R_0402_1005Metric, F.Cu at (20.6, 63.1)
- added R113: 4.7k, Resistor_SMD:R_0402_1005Metric, F.Cu at (20.6, 65.1)
- added R114: 4.7k, Resistor_SMD:R_0402_1005Metric, F.Cu at (20.6, 67.1)
- added R115: 4.7k, Resistor_SMD:R_0402_1005Metric, F.Cu at (23.5, 55.1)
- added R116: 4.7k, Resistor_SMD:R_0402_1005Metric, F.Cu at (23.5, 57.1)
- added R117: 4.7k, Resistor_SMD:R_0402_1005Metric, F.Cu at (23.5, 59.1)
- added R118: 4.7k, Resistor_SMD:R_0402_1005Metric, F.Cu at (23.5, 61.1)
- added R119: 22R, Resistor_SMD:R_0402_1005Metric, F.Cu at (80.1, 29.6)
- added R120: 22R, Resistor_SMD:R_0402_1005Metric, F.Cu at (83.0, 17.7)
- added R121: 22R, Resistor_SMD:R_0402_1005Metric, F.Cu at (83.0, 19.7)
- added R122: 22R, Resistor_SMD:R_0402_1005Metric, F.Cu at (83.0, 21.6)
- added R123: 22R, Resistor_SMD:R_0402_1005Metric, F.Cu at (83.0, 23.6)
- added R124: 22R, Resistor_SMD:R_0402_1005Metric, F.Cu at (83.0, 25.6)
- added R125: 22R, Resistor_SMD:R_0402_1005Metric, F.Cu at (83.0, 27.6)
- added R126: 22R, Resistor_SMD:R_0402_1005Metric, F.Cu at (83.0, 29.6)
- added R127: 22R, Resistor_SMD:R_0402_1005Metric, F.Cu at (85.9, 17.7)
- added R128: 22R, Resistor_SMD:R_0402_1005Metric, F.Cu at (85.9, 19.7)
- added R129: 22R, Resistor_SMD:R_0402_1005Metric, F.Cu at (85.9, 21.6)
- added R130: 22R, Resistor_SMD:R_0402_1005Metric, F.Cu at (85.9, 23.6)
- added R93: 10k, Resistor_SMD:R_0402_1005Metric, F.Cu at (80.1, 17.7)
- added REF**: M.2 EC Board, M.2-EC-Board:M.2 EC Board, F.Cu at (175.1, 225.2)
- added U2: SI52147-A01AGM, SI52147_A01AGM:QFN15.75P236X236X100-48_SKY-L, F.Cu at (209.5, 137.6)
- moved H4 306.8 mm to (321.0, 232.5)
- moved H2 260.2 mm to (321.0, 100.0)
- moved H3 209.2 mm to (163.0, 232.5)
- moved H1 103.4 mm to (163.2, 77.1)
- moved R94 71.3 mm to (50.7, 84.9)
- moved R96 71.3 mm to (50.7, 88.9)
- moved R95 71.3 mm to (50.7, 86.9)
- moved R99 67.2 mm to (52.0, 91.5)
- moved R100 64.7 mm to (53.6, 88.9)
- moved R97 64.7 mm to (53.6, 84.9)
- moved R98 64.7 mm to (53.6, 86.9)
- moved C198 64.3 mm to (32.7, 44.2)
- moved C211 60.9 mm to (47.0, 18.3)
- moved C213 60.9 mm to (47.0, 25.0)
- moved C214 60.9 mm to (47.0, 28.4)
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Connections:
- C201 pad 1: PCIE_NVME_CLKP -> PCIE_NVME1_CLKP
- C202 pad 1: PCIE_NVME_CLKN -> PCIE_NVME1_CLKN
- C203 pad 1: PCIE_NVME_CLKP -> PCIE_NVME0_CLKP
- C204 pad 1: PCIE_NVME_CLKN -> PCIE_NVME0_CLKN
- CN1 pad A10: 3V3 -> PCIE_3V3
- CN1 pad A9: 3V3 -> PCIE_3V3
- CN1 pad B8: 3V3 -> PCIE_3V3
- R53 pad 1: 3V3 -> PCIE_3V3
- R54 pad 1: 3V3 -> PCIE_3V3
- R59 pad 1: PCIE_3V3_STANDBY -> 3V3_STBY
- U5 pad AA29: unconnected-(U5C-CAN_TX0/PEU1_LINKUP1-PadAA29) -> FT_CAN_TXD0
- U5 pad AB27: unconnected-(U5C-UART_0_DTR_N/GPIO0_A6-PadAB27) -> FT_UART_0_DTR_N
- U5 pad AB28: unconnected-(U5C-QSPI_WP_IO2-PadAB28) -> FT_QSPI_IO2
- U5 pad AB29: unconnected-(U5C-PEU1_LINKUP0/GPIO0_A7/SCI-PadAB29) -> FT_PEU1_LINKUP0
- U5 pad AB30: unconnected-(U5C-RSVD16_DOWN-PadAB30) -> GND
- U5 pad AC27: unconnected-(U5C-UART_0_RTS_N/GPIO0_A5-PadAC27) -> FT_UART_0_RTS_N
- U5 pad AC28: unconnected-(U5C-RSVD3_UP-PadAC28) -> VDD_IO
- U5 pad AD13: unconnected-(U5C-FT_RSVD11-PadAD13) -> FT_HDA_SDI0
- U5 pad AD14: unconnected-(U5C-FT_RSVD5-PadAD14) -> FT_LPC_IRQ_N
- U5 pad AD15: unconnected-(U5C-SD_CMD/GPIO1_B1-PadAD15) -> FT_SD_CMD
- U5 pad AD16: unconnected-(U5C-UART_0_RXD-PadAD16) -> FT_UART_0_RXD
- U5 pad AD26: unconnected-(U5C-SD_DAT2/GPIO1_B5-PadAD26) -> FT_SD_DATA2
- U5 pad AD27: unconnected-(U5C-SD_DETECT-PadAD27) -> FT_SD_DETECT
- U5 pad AD28: (no net) -> FT_LPC_LAD3
- U5 pad AD29: unconnected-(U5C-QSPI_CSN1/GPIO1_B7-PadAD29) -> FT_QSPI_CSN1
- U5 pad AE11: unconnected-(U5C-SPI0_SCK/GPIO1_A6-PadAE11) -> FT_SPI0_SCK
- U5 pad AE12: unconnected-(U5C-FT_RSVD7/GPIO1_A3-PadAE12) -> FT_LPC_LAD0
- U5 pad AE13: unconnected-(U5C-RSVD23_DOWN-PadAE13) -> Net-(U5C-RSVD23_DOWN)
- U5 pad AE14: unconnected-(U5C-RSVD8_DOWN-PadAE14) -> GND
- U5 pad AE16: unconnected-(U5C-FT_RSVD0-PadAE16) -> FT_LPC_CLK
- U5 pad AE17: unconnected-(U5C-TCK_SWJ-PadAE17) -> Net-(U5C-TCK_SWJ)
- U5 pad AE18: unconnected-(U5C-FT_RSVD4-PadAE18) -> FT_LPC_LFRAME_N
- U5 pad AE19: unconnected-(U5C-FT_RSVD3-PadAE19) -> FT_LPC_RSTN
- U5 pad AE20: unconnected-(U5C-FT_RSVD14-PadAE20) -> FT_HDA_RST
- U5 pad AE21: unconnected-(U5C-SD_DAT1/GPIO1_B4-PadAE21) -> FT_SD_DATA1
- U5 pad AE22: unconnected-(U5C-SD_CLK/GPIO1_B2-PadAE22) -> FT_SD_CLK
- U5 pad AE23: unconnected-(U5C-FT_RSVD15-PadAE23) -> FT_HDA_SYNC
- U5 pad AE24: unconnected-(U5C-FT_RSVD9/SPI1_CSN_3-PadAE24) -> FT_LPC_LAD2
- U5 pad AE25: unconnected-(U5C-FT_RSVD12-PadAE25) -> FT_HDA_SDO
- U5 pad AE28: unconnected-(U5C-UART_0_TXD-PadAE28) -> FT_UART_0_TXD
- U5 pad AE29: unconnected-(U5C-UART_1_TXD-PadAE29) -> FT_UART_1_TXD
- U5 pad AF10: unconnected-(U5C-SPI0_CSN0/GPIO1_A5-PadAF10) -> FT_SPI0_CSN0
- U5 pad AF14: unconnected-(U5C-UART_1_RXD-PadAF14) -> FT_UART_1_RXD
- U5 pad AF16: unconnected-(U5C-I2C0_SDA-PadAF16) -> FT_I2C_0_SDA
- U5 pad AF17: unconnected-(U5C-SPI0_SO/GPIO1_A7-PadAF17) -> FT_SPI0_SO
- U5 pad AF18: unconnected-(U5C-FT_RSVD8/GPIO1_A4-PadAF18) -> FT_LPC_LAD1
- U5 pad AF19: unconnected-(U5C-UART_3_RXD/SPI1_SO/FT_RSVD18-PadAF19) -> Net-(U5C-UART_3_RXD/SPI1_SO/HDA_SDI2)
- U5 pad AF20: unconnected-(U5C-FT_RSVD13-PadAF20) -> FT_HDA_BCLK
- U5 pad AF21: unconnected-(U5C-RSVD24_DOWN-PadAF21) -> GND
- U5 pad AF23: unconnected-(U5C-UART_2_RXD/SPI1_CSN0/GPIO0_B5-PadAF23) -> Net-(U5C-UART_2_RXD/SPI1_CSN0/GPIO0_B5)
- U5 pad AF24: unconnected-(U5C-SD_DAT3/GPIO1_B6-PadAF24) -> FT_SD_DATA3
- U5 pad AF25: unconnected-(U5C-FT_RSVD6-PadAF25) -> FT_LPC_LDRQ_N
- U5 pad AF28: unconnected-(U5C-SD_DAT0/GPIO1_B3-PadAF28) -> FT_SD_DATA0
- U5 pad AG15: unconnected-(U5C-SPI0_SI/GPIO1_B0-PadAG15) -> FT_SPI0_SI
- U5 pad AG18: unconnected-(U5C-I2C0_SCL-PadAG18) -> FT_I2C_0_SCL
- U5 pad AG19: unconnected-(U5C-CAN_RXD2/I2C2_SDA/TDO_SWJ-PadAG19) -> Net-(U5C-CAN_RXD2/I2C2_SDA/TDO_SWJ)
- U5 pad H15: unconnected-(U5C-UART_0_DSR_N/GPIO0_A3-PadH15) -> FT_UART_0_DSR_N
- U5 pad H18: unconnected-(U5C-RSVD6_UP-PadH18) -> VDD_IO
- U5 pad H19: unconnected-(U5C-RSVD4_UP-PadH19) -> VDD_IO
- U5 pad H9: unconnected-(U5D-RGMII1_MDC-PadH9) -> FT_GMAC1_MDC
- U5 pad J10: unconnected-(U5D-RGMII0_RX_CTL-PadJ10) -> FT_GMAC0_RX_CTL
- U5 pad J11: unconnected-(U5D-RGMII0_RXD2-PadJ11) -> FT_GMAC0_RXD2
- U5 pad J12: unconnected-(U5D-RGMII0_RXD0-PadJ12) -> FT_GMAC0_RXD1
- U5 pad J13: unconnected-(U5D-RGMII0_TXD3-PadJ13) -> RGMII0_TXD3
- U5 pad J14: unconnected-(U5D-RGMII0_TXD0-PadJ14) -> RGMII0_TXD0
- U5 pad J15: unconnected-(U5D-RGMII0_TXD2-PadJ15) -> RGMII0_TXD2
- U5 pad J16: unconnected-(U5C-CAN_TXD1/PEU1_LINKUP2/NTRST_SWJ-PadJ16) -> FT_CAN_TXD1
- U5 pad J17: unconnected-(U5C-UART_0_DCD_N/GPIO0_A2-PadJ17) -> FT_UART_0_DCD_N
- U5 pad J18: unconnected-(U5C-CPI_RST_OK-PadJ18) -> FT_CRU_RST_OK
- U5 pad J19: unconnected-(U5C-CAN_RXD1/I2C2_SCL/SWDO_SWJ-PadJ19) -> FT_CAN_RXD1
- U5 pad J21: unconnected-(U5D-RGMII9_MDIO-PadJ21) -> FT_GMAC1_MDIO
- U5 pad J24: unconnected-(U5C-RSVD14_DOWN-PadJ24) -> GND
- U5 pad J25: unconnected-(U5C-RSVD13_DOWN-PadJ25) -> GND
- U5 pad K10: unconnected-(U5D-RGMII1_RX_CLK-PadK10) -> FT_GMAC1_RX_CLK
- U5 pad K11: unconnected-(U5D-RGMII1_TXD1/SPI0_CSN1-PadK11) -> RGMII1_TXD1
- U5 pad K12: (no net) -> FT_GMAC0_RXD0
- U5 pad K13: unconnected-(U5D-RGMII0_GTX_CLK-PadK13) -> RGMII0_GTX_CLK
- U5 pad K14: unconnected-(U5D-RGMII0_TXD1-PadK14) -> RGMII0_TXD1
- U5 pad K15: unconnected-(U5D-RGMII0_TX_CTL-PadK15) -> RGMII0_TX_CTL
- U5 pad K16: unconnected-(U5C-CAN_RXD0/SWDITMS_SWJ-PadK16) -> FT_CAN_RXD0
- U5 pad K17: unconnected-(U5C-UART_0_CTS_N/GPIO0_A1-PadK17) -> FT_UART_0_CTS_N
- U5 pad K18: unconnected-(U5D-RGMII0_MDC-PadK18) -> FT_GMAC0_MDC
- U5 pad K19: unconnected-(U5C-RSVD7_DOWN-PadK19) -> Net-(U5C-RSVD7_DOWN)
- U5 pad K20: unconnected-(U5C-POR_N-PadK20) -> FT_POR_N
- U5 pad K21: unconnected-(U5C-UART_0_RI_N/GPIO0_A4-PadK21) -> FT_UART_0_RI_N
- U5 pad K22: unconnected-(U5D-RGMII0_MDIO-PadK22) -> FT_GMAC0_MDIO
- U5 pad K24: unconnected-(U5C-PEU0_LINKUP1-PadK24) -> FT_PEU0_LINKUP1
- U5 pad K25: unconnected-(U5C-PEU0_LINKUP0-PadK25) -> FT_PEU0_LINKUP0
- U5 pad K28: unconnected-(U5C-RSVD10_DOWN-PadK28) -> GND
- U5 pad K9: unconnected-(U5D-RGMII1_RX_CTL/GPIO1_A1-PadK9) -> FT_GMAC1_RX_CTL
- U5 pad L10: unconnected-(U5D-RGMII1_GTX_CLK-PadL10) -> RGMII1_TXD2
- U5 pad L11: (no net) -> RGMII1_GTX_CLK
- U5 pad L12: unconnected-(U5D-RGMII0_RXD3-PadL12) -> FT_GMAC0_RXD3
- U5 pad L13: unconnected-(U5D-RGMII0_RX_CLK-PadL13) -> FT_GMAC0_RX_CLK
- U5 pad L14: unconnected-(U5C-ALL_PLL_LOCK/I2C_1_SDL-PadL14) -> FT_I2C_1_SCL
- U5 pad L15: unconnected-(U5C-CRU_CLK_OBV/I2C_1_SDA/GPIO_A0-PadL15) -> FT_I2C_1_SDA
- U5 pad L29: unconnected-(U5C-RSVD15_DOWN-PadL29) -> GND
- U5 pad M10: unconnected-(U5D-RGMII1_TX_CTL/GPIO0_B4-PadM10) -> RGMII1_TX_CTL
- U5 pad M11: unconnected-(U5D-RGMII1_TXD0/GPIO1_A2-PadM11) -> RGMII1_TXD0
- U5 pad M26: unconnected-(U5C-RSVD18_DOWN-PadM26) -> GND
- U5 pad M9: unconnected-(U5D-RGMII1_RXD3/GPIO1_A0-PadM9) -> FT_GMAC1_RXD3
- U5 pad N10: unconnected-(U5D-RGMII1_RXD2/GPIO0_B2-PadN10) -> FT_GMAC1_RXD2
- U5 pad N11: unconnected-(U5D-RGMII1_TXD3/GPIO0_B3-PadN11) -> RGMII1_TXD3
- U5 pad N26: unconnected-(U5C-PEU0_LINKUP2-PadN26) -> FT_PEU0_LINKUP2
- U5 pad N28: unconnected-(U5C-RSVD9_DOWN-PadN28) -> GND
- U5 pad N29: unconnected-(U5C-RSVD17_DOWN-PadN29) -> GND
- U5 pad P10: unconnected-(U5D-RGMII1_RXD0/GPIO0_B0-PadP10) -> FT_GMAC1_RXD0
- U5 pad P26: unconnected-(U5C-RSVD19_DOWN-PadP26) -> GND
- U5 pad P27: unconnected-(U5C-CLK_REF-PadP27) -> FT_CLK_REF_48M
- U5 pad P28: unconnected-(U5C-RSVD21_DOWN-PadP28) -> GND
- U5 pad P29: unconnected-(U5C-RSVD0_UP-PadP29) -> VDD_IO
- U5 pad P9: unconnected-(U5D-RGMII1_RXD1/GPIO0_B1-PadP9) -> FT_GMAC1_RXD1
- U5 pad R27: unconnected-(U5C-QSPI_SCK-PadR27) -> FT_QSPI_SCK
- U5 pad R29: unconnected-(U5C-PWR_CTR1-PadR29) -> FT_PWR_CTR1
- U5 pad T26: unconnected-(U5C-PWR_CTR0-PadT26) -> FT_PWR_CTR0
- U5 pad T27: unconnected-(U5C-RSVD20_DOWN-PadT27) -> GND
- U5 pad T28: unconnected-(U5C-RSVD12_DOWN-PadT28) -> GND
- U5 pad T29: unconnected-(U5C-RSVD22_DOWN-PadT29) -> GND
- U5 pad U26: unconnected-(U5C-QSPI_HOLD_IO3-PadU26) -> FT_QSPI_IO3
- U5 pad U27: unconnected-(U5C-QSPI_CSN0-PadU27) -> FT_QSPI_CSN0
- U5 pad U29: unconnected-(U5C-RSVD1_UP-PadU29) -> VDD_IO
- U5 pad V29: unconnected-(U5C-RSVD2_UP-PadV29) -> VDD_IO
- U5 pad W27: unconnected-(U5C-RSVD11_DOWN-PadW27) -> GND
- U5 pad W28: unconnected-(U5C-QSPI_SO_IO0-PadW28) -> FT_QSPI_IO0
- U5 pad W29: unconnected-(U5C-RSVD5_UP-PadW29) -> VDD_IO
- U5 pad Y28: unconnected-(U5C-QSPI_SI_IO1-PadY28) -> FT_QSPI_IO1
Routing:
- net FT_PEU1_TXP15: track 95.8 -> 0.00 mm
- net FT_PEU1_TXP14: track 94.9 -> 0.00 mm
- net FT_PEU1_RXN15: track 100.5 -> 5.97 mm
- net FT_PEU1_TXN15: track 94.3 -> 0.00 mm
- net FT_PEU1_TXN14: track 93.2 -> 0.00 mm
- net FT_PEU1_RXP15: track 99.8 -> 6.97 mm
- net FT_PEU1_RXN14: track 90.5 -> 0.00 mm
- net FT_PEU1_RXN13: track 89.2 -> 0.00 mm
- net FT_PEU1_RXP14: track 88.8 -> 0.00 mm
- net FT_PEU1_RXP13: track 87.6 -> 0.00 mm
